Commit message: new urdf file

File: install/robot_pkg/share/robot_pkg/urdf/TTR01.urdf.xacro (robot description, xacro)
@@ -1,594 +1 @@
-<?xml version="1.0" encoding="utf-8"?>
-<!-- This URDF was automatically created by SolidWorks to URDF Exporter! Originally created by Stephen Brawner (brawner@gmail.com)
-     Commit Version: 1.6.0-4-g7f85cfe  Build Version: 1.6.7995.38578
-     For more information, please see http://wiki.ros.org/sw_urdf_exporter -->
-<robot xmlns:xacro="http://www.ros.org/wiki/xacro" name="TTR01">
-  <link
-    name="base_link">
-    <inertial>
-      <origin
-        xyz="0.00041344 3.7856E-10 -0.018281"
-        rpy="0 0 0" />
-      <mass
-        value="0.68825" />
-      <inertia
-        ixx="0.00041167"
-        ixy="-1.1043E-10"
-        ixz="-2.4196E-06"
-        iyy="0.00052928"
-        iyz="7.1835E-12"
-        izz="0.00085508" />
-    </inertial>
-    <visual>
-      <origin
-        xyz="0 0 0"
-        rpy="0 0 0" />
-      <geometry>
-        <mesh
-          filename="package://robot_pkg/meshes/base_link.STL" />
-      </geometry>
-      <material
-        name="">
-        <color
-          rgba="1 1 1 1" />
-      </material>
-    </visual>
-    <collision>
-      <origin
-        xyz="0 0 0"
-        rpy="0 0 0" />
-      <geometry>
-        <mesh
-          filename="package://robot_pkg/meshes/base_link.STL" />
-      </geometry>
-    </collision>
-  </link>
-  <link
-    name="L_wheel_link">
-    <inertial>
-      <origin
-        xyz="-5.629E-10 5.4357E-10 -0.015886"
-        rpy="0 0 0" />
-      <mass
-        value="0.048724" />
-      <inertia
-        ixx="1.5816E-05"
-        ixy="4.1458E-09"
-        ixz="-1.7893E-13"
-        iyy="1.5814E-05"
-        iyz="1.7858E-13"
-        izz="2.6155E-05" />
-    </inertial>
-    <visual>
-      <origin
-        xyz="0 0 0"
-        rpy="0 0 0" />
-      <geometry>
-        <mesh
-          filename="package://robot_pkg/meshes/L_wheel_link.STL" />
-      </geometry>
-      <material
-        name="">
-        <color
-          rgba="0.75294 0.75294 0.75294 1" />
-      </material>
-    </visual>
-    <collision>
-      <origin
-        xyz="0 0 0"
-        rpy="0 0 0" />
-      <geometry>
-        <mesh
-          filename="package://robot_pkg/meshes/L_wheel_link.STL" />
-      </geometry>
-    </collision>
-  </link>
-  <joint
-    name="L_wheel_joint"
-    type="continuous">
-    <origin
-      xyz="0 -0.071 -0.0225"
-      rpy="-1.5708 0 0" />
-    <parent
-      link="base_link" />
-    <child
-      link="L_wheel_link" />
-    <axis
-      xyz="0 0 1" />
-    <limit
-      effort="0.323"
-      velocity="10.47" />
-  </joint>
-  <link
-    name="R_wheel_link">
-    <inertial>
-      <origin
-        xyz="-4.8323E-10 -6.1547E-10 0.015886"
-        rpy="0 0 0" />
-      <mass
-        value="0.048724" />
-      <inertia
-        ixx="1.5817E-05"
-        ixy="-3.7851E-09"
-        ixz="1.5281E-13"
-        iyy="1.5813E-05"
-        iyz="2.0138E-13"
-        izz="2.6155E-05" />
-    </inertial>
-    <visual>
-      <origin
-        xyz="0 0 0"
-        rpy="0 0 0" />
-      <geometry>
-        <mesh
-          filename="package://robot_pkg/meshes/R_wheel_link.STL" />
-      </geometry>
-      <material
-        name="">
-        <color
-          rgba="0.75294 0.75294 0.75294 1" />
-      </material>
-    </visual>
-    <collision>
-      <origin
-        xyz="0 0 0"
-        rpy="0 0 0" />
-      <geometry>
-        <mesh
-          filename="package://robot_pkg/meshes/R_wheel_link.STL" />
-      </geometry>
-    </collision>
-  </link>
-  <joint
-    name="R_wheel_joint"
-    type="continuous">
-    <origin
-      xyz="0 0.071 -0.0225"
-      rpy="-1.5708 0 0" />
-    <parent
-      link="base_link" />
-    <child
-      link="R_wheel_link" />
-    <axis
-      xyz="0 0 1" />
-    <limit
-      effort="0.323"
-      velocity="10.47" />
-  </joint>
-  <link
-    name="U_base_wheel_1_link">
-    <inertial>
-      <origin
-        xyz="0.0041491 -8.4566E-05 0.0063957"
-        rpy="0 0 0" />
-      <mass
-        value="0.009087" />
-      <inertia
-        ixx="5.254E-07"
-        ixy="-4.3301E-10"
-        ixz="-9.4848E-08"
-        iyy="4.8759E-07"
-        iyz="1.0854E-09"
-        izz="7.6419E-07" />
-    </inertial>
-    <visual>
-      <origin
-        xyz="0 0 0"
-        rpy="0 0 0" />
-      <geometry>
-        <mesh
-          filename="package://robot_pkg/meshes/U_base_wheel_1_link.STL" />
-      </geometry>
-      <material
-        name="">
-        <color
-          rgba="0.77647 0.75686 0.73725 1" />
-      </material>
-    </visual>
-    <collision>
-      <origin
-        xyz="0 0 0"
-        rpy="0 0 0" />
-      <geometry>
-        <mesh
-          filename="package://robot_pkg/meshes/U_base_wheel_1_link.STL" />
-      </geometry>
-    </collision>
-  </link>
-  <joint
-    name="U_base_wheel_1_joint"
-    type="continuous">
-    <origin
-      xyz="0.057514 0 -0.0234"
-      rpy="3.1416 0 0" />
-    <parent
-      link="base_link" />
-    <child
-      link="U_base_wheel_1_link" />
-    <axis
-      xyz="0 0 -1" />
-    <limit
-      effort="0.323"
-      velocity="10.47" />
-  </joint>
-  <link
-    name="U_wheel_1_link">
-    <inertial>
-      <origin
-        xyz="-0.0015 0 0"
-        rpy="0 0 0" />
-      <mass
-        value="0.0045951" />
-      <inertia
-        ixx="2.7312E-07"
-        ixy="-2.3056E-23"
-        ixz="-2.2711E-23"
-        iyy="2.7312E-07"
-        iyz="-9.4919E-23"
-        izz="4.0127E-07" />
-    </inertial>
-    <visual>
-      <origin
-        xyz="0 0 0"
-        rpy="0 0 0" />
-      <geometry>
-        <mesh
-          filename="package://robot_pkg/meshes/U_wheel_1_link.STL" />
-      </geometry>
-      <material
-        name="">
-        <color
-          rgba="1 1 1 1" />
-      </material>
-    </visual>
-    <collision>
-      <origin
-        xyz="0 0 0"
-        rpy="0 0 0" />
-      <geometry>
-        <mesh
-          filename="package://robot_pkg/meshes/U_wheel_1_link.STL" />
-      </geometry>
-    </collision>
-  </link>
-  <joint
-    name="U_wheel_1_joint"
-    type="continuous">
-    <origin
-      xyz="0.015768 -0.00018037 0.022119"
-      rpy="1.5822 -1.5708 0" />
-    <parent
-      link="U_base_wheel_1_link" />
-    <child
-      link="U_wheel_1_link" />
-    <axis
-      xyz="0 0 1" />
-    <limit
-      effort="0.323"
-      velocity="10.47" />
-  </joint>
-  <link
-    name="U_base_wheel_2_link">
-    <inertial>
-      <origin
-        xyz="-0.0041491 8.4566E-05 0.00049565"
-        rpy="0 0 0" />
-      <mass
-        value="0.009087" />
-      <inertia
-        ixx="5.254E-07"
-        ixy="-4.3301E-10"
-        ixz="9.4848E-08"
-        iyy="4.8759E-07"
-        iyz="-1.0854E-09"
-        izz="7.6419E-07" />
-    </inertial>
-    <visual>
-      <origin
-        xyz="0 0 0"
-        rpy="0 0 0" />
-      <geometry>
-        <mesh
-          filename="package://robot_pkg/meshes/U_base_wheel_2_link.STL" />
-      </geometry>
-      <material
-        name="">
-        <color
-          rgba="0.77647 0.75686 0.73725 1" />
-      </material>
-    </visual>
-    <collision>
-      <origin
-        xyz="0 0 0"
-        rpy="0 0 0" />
-      <geometry>
-        <mesh
-          filename="package://robot_pkg/meshes/U_base_wheel_2_link.STL" />
-      </geometry>
-    </collision>
-  </link>
-  <joint
-    name="U_base_wheel_2_joint"
-    type="continuous">
-    <origin
-      xyz="-0.057514 0 -0.0293"
-      rpy="3.1416 0 0" />
-    <parent
-      link="base_link" />
-    <child
-      link="U_base_wheel_2_link" />
-    <axis
-      xyz="0 0 -1" />
-    <limit
-      effort="0.323"
-      velocity="10.47" />
-  </joint>
-  <link
-    name="U_wheel_2_link">
-    <inertial>
-      <origin
-        xyz="-0.0015 0 -8.6736E-19"
-        rpy="0 0 0" />
-      <mass
-        value="0.0045951" />
-      <inertia
-        ixx="2.7312E-07"
-        ixy="4.1047E-23"
-        ixz="1.9175E-23"
-        iyy="2.7312E-07"
-        iyz="-7.2378E-23"
-        izz="4.0127E-07" />
-    </inertial>
-    <visual>
-      <origin
-        xyz="0 0 0"
-        rpy="0 0 0" />
-      <geometry>
-        <mesh
-          filename="package://robot_pkg/meshes/U_wheel_2_link.STL" />
-      </geometry>
-      <material
-        name="">
-        <color
-          rgba="1 1 1 1" />
-      </material>
-    </visual>
-    <collision>
-      <origin
-        xyz="0 0 0"
-        rpy="0 0 0" />
-      <geometry>
-        <mesh
-          filename="package://robot_pkg/meshes/U_wheel_2_link.STL" />
-      </geometry>
-    </collision>
-  </link>
-  <joint
-    name="U_wheel_2_joint"
-    type="continuous">
-    <origin
-      xyz="-0.015768 0.00018037 0.016219"
-      rpy="1.5822 -1.5708 0" />
-    <parent
-      link="U_base_wheel_2_link" />
-    <child
-      link="U_wheel_2_link" />
-    <axis
-      xyz="0 0 1" />
-    <limit
-      effort="0.323"
-      velocity="10.47" />
-  </joint>
-  <link
-    name="Support_A_link">
-    <inertial>
-      <origin
-        xyz="0 0 0"
-        rpy="0 0 0" />
-      <mass
-        value="0" />
-      <inertia
-        ixx="0"
-        ixy="0"
-        ixz="0"
-        iyy="0"
-        iyz="0"
-        izz="0" />
-    </inertial>
-    <visual>
-      <origin
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
Commit message: gazebo file

File: install/robot_pkg/share/robot_pkg/urdf/TTR01.urdf.xacro (robot description, xacro)
@@ -1 +1,595 @@
-/home/ttrxx/TTRXX_WS/build/robot_pkg/urdf/TTR01.urdf.xacro
+<?xml version="1.0" ?>
+<!-- This URDF was automatically created by SolidWorks to URDF Exporter! Originally created by Stephen Brawner (brawner@gmail.com)
+     Commit Version: 1.6.0-4-g7f85cfe  Build Version: 1.6.7995.38578
+     For more information, please see http://wiki.ros.org/sw_urdf_exporter -->
+<robot xmlns:xacro="http://www.ros.org/wiki/xacro" name="TTR01">
+  <link
+    name="base_link">
+    <inertial>
+      <origin
+        xyz="0.00041344 3.7856E-10 -0.018281"
+        rpy="0 0 0" />
+      <mass
+        value="0.68825" />
+      <inertia
+        ixx="0.00041167"
+        ixy="-1.1043E-10"
+        ixz="-2.4196E-06"
+        iyy="0.00052928"
+        iyz="7.1835E-12"
+        izz="0.00085508" />
+    </inertial>
+    <visual>
+      <origin
+        xyz="0 0 0"
+        rpy="0 0 0" />
+      <geometry>
+        <mesh
+          filename="package://robot_pkg/meshes/base_link.STL" />
+      </geometry>
+      <material
+        name="">
+        <color
+          rgba="1 1 1 1" />
+      </material>
+    </visual>
+    <collision>
+      <origin
+        xyz="0 0 0"
+        rpy="0 0 0" />
+      <geometry>
+        <mesh
+          filename="package://robot_pkg/meshes/base_link.STL" />
+      </geometry>
+    </collision>
+  </link>
+  <link
+    name="L_wheel_link">
+    <inertial>
+      <origin
+        xyz="-5.629E-10 5.4357E-10 -0.015886"
+        rpy="0 0 0" />
+      <mass
+        value="0.048724" />
+      <inertia
+        ixx="1.5816E-05"
+        ixy="4.1458E-09"
+        ixz="-1.7893E-13"
+        iyy="1.5814E-05"
+        iyz="1.7858E-13"
+        izz="2.6155E-05" />
+    </inertial>
+    <visual>
+      <origin
+        xyz="0 0 0"
+        rpy="0 0 0" />
+      <geometry>
+        <mesh
+          filename="package://robot_pkg/meshes/L_wheel_link.STL" />
+      </geometry>
+      <material
+        name="">
+        <color
+          rgba="0.75294 0.75294 0.75294 1" />
+      </material>
+    </visual>
+    <collision>
+      <origin
+        xyz="0 0 0"
+        rpy="0 0 0" />
+      <geometry>
+        <mesh
+          filename="package://robot_pkg/meshes/L_wheel_link.STL" />
+      </geometry>
+    </collision>
+  </link>
+  <joint
+    name="L_wheel_joint"
+    type="continuous">
+    <origin
+      xyz="0 -0.071 -0.0225"
+      rpy="-1.5708 0 0" />
+    <parent
+      link="base_link" />
+    <child
+      link="L_wheel_link" />
+    <axis
+      xyz="0 0 1" />
+    <limit
+      effort="0.323"
+      velocity="10.47" />
+  </joint>
+  <link
+    name="R_wheel_link">
+    <inertial>
+      <origin
+        xyz="-4.8323E-10 -6.1547E-10 0.015886"
+        rpy="0 0 0" />
+      <mass
+        value="0.048724" />
+      <inertia
+        ixx="1.5817E-05"
+        ixy="-3.7851E-09"
+        ixz="1.5281E-13"
+        iyy="1.5813E-05"
+        iyz="2.0138E-13"
+        izz="2.6155E-05" />
+    </inertial>
+    <visual>
+      <origin
+        xyz="0 0 0"
+        rpy="0 0 0" />
+      <geometry>
+        <mesh
+          filename="package://robot_pkg/meshes/R_wheel_link.STL" />
+      </geometry>
+      <material
+        name="">
+        <color
+          rgba="0.75294 0.75294 0.75294 1" />
+      </material>
+    </visual>
+    <collision>
+      <origin
+        xyz="0 0 0"
+        rpy="0 0 0" />
+      <geometry>
+        <mesh
+          filename="package://robot_pkg/meshes/R_wheel_link.STL" />
+      </geometry>
+    </collision>
+  </link>
+  <joint
+    name="R_wheel_joint"
+    type="continuous">
+    <origin
+      xyz="0 0.071 -0.0225"
+      rpy="-1.5708 0 0" />
+    <parent
+      link="base_link" />
+    <child
+      link="R_wheel_link" />
+    <axis
+      xyz="0 0 1" />
+    <limit
+      effort="0.323"
+      velocity="10.47" />
+  </joint>
+  <link
+    name="U_base_wheel_1_link">
+    <inertial>
+      <origin
+        xyz="0.0041491 -8.4566E-05 0.0063957"
+        rpy="0 0 0" />
+      <mass
+        value="0.009087" />
+      <inertia
+        ixx="5.254E-07"
+        ixy="-4.3301E-10"
+        ixz="-9.4848E-08"
+        iyy="4.8759E-07"
+        iyz="1.0854E-09"
+        izz="7.6419E-07" />
+    </inertial>
+    <visual>
+      <origin
+        xyz="0 0 0"
+        rpy="0 0 0" />
+      <geometry>
+        <mesh
+          filename="package://robot_pkg/meshes/U_base_wheel_1_link.STL" />
+      </geometry>
+      <material
+        name="">
+        <color
+          rgba="0.77647 0.75686 0.73725 1" />
+      </material>
+    </visual>
+    <collision>
+      <origin
+        xyz="0 0 0"
+        rpy="0 0 0" />
+      <geometry>
+        <mesh
+          filename="package://robot_pkg/meshes/U_base_wheel_1_link.STL" />
+      </geometry>
+    </collision>
+  </link>
+  <joint
+    name="U_base_wheel_1_joint"
+    type="continuous">
+    <origin
+      xyz="0.057514 0 -0.0234"
+      rpy="3.1416 0 0" />
+    <parent
+      link="base_link" />
+    <child
+      link="U_base_wheel_1_link" />
+    <axis
+      xyz="0 0 -1" />
+    <limit
+      effort="0.323"
+      velocity="10.47" />
+  </joint>
+  <link
+    name="U_wheel_1_link">
+    <inertial>
+      <origin
+        xyz="-0.0015 0 0"
+        rpy="0 0 0" />
+      <mass
+        value="0.0045951" />
+      <inertia
+        ixx="2.7312E-07"
+        ixy="-2.3056E-23"
+        ixz="-2.2711E-23"
+        iyy="2.7312E-07"
+        iyz="-9.4919E-23"
+        izz="4.0127E-07" />
+    </inertial>
+    <visual>
+      <origin
+        xyz="0 0 0"
+        rpy="0 0 0" />
+      <geometry>
+        <mesh
+          filename="package://robot_pkg/meshes/U_wheel_1_link.STL" />
+      </geometry>
+      <material
+        name="">
+        <color
+          rgba="1 1 1 1" />
+      </material>
+    </visual>
+    <collision>
+      <origin
+        xyz="0 0 0"
+        rpy="0 0 0" />
+      <geometry>
+        <mesh
+          filename="package://robot_pkg/meshes/U_wheel_1_link.STL" />
+      </geometry>
+    </collision>
+  </link>
+  <joint
+    name="U_wheel_1_joint"
+    type="continuous">
+    <origin
+      xyz="0.015768 -0.00018037 0.022119"
+      rpy="1.5822 -1.5708 0" />
+    <parent
+      link="U_base_wheel_1_link" />
+    <child
+      link="U_wheel_1_link" />
+    <axis
+      xyz="0 0 1" />
+    <limit
+      effort="0.323"
+      velocity="10.47" />
+  </joint>
+  <link
+    name="U_base_wheel_2_link">
+    <inertial>
+      <origin
+        xyz="-0.0041491 8.4566E-05 0.00049565"
+        rpy="0 0 0" />
+      <mass
+        value="0.009087" />
+      <inertia
+        ixx="5.254E-07"
+        ixy="-4.3301E-10"
+        ixz="9.4848E-08"
+        iyy="4.8759E-07"
+        iyz="-1.0854E-09"
+        izz="7.6419E-07" />
+    </inertial>
+    <visual>
+      <origin
+        xyz="0 0 0"
+        rpy="0 0 0" />
+      <geometry>
+        <mesh
+          filename="package://robot_pkg/meshes/U_base_wheel_2_link.STL" />
+      </geometry>
+      <material
+        name="">
+        <color
+          rgba="0.77647 0.75686 0.73725 1" />
+      </material>
+    </visual>
+    <collision>
+      <origin
+        xyz="0 0 0"
+        rpy="0 0 0" />
+      <geometry>
+        <mesh
+          filename="package://robot_pkg/meshes/U_base_wheel_2_link.STL" />
+      </geometry>
+    </collision>
+  </link>
+  <joint
+    name="U_base_wheel_2_joint"
+    type="continuous">
+    <origin
+      xyz="-0.057514 0 -0.0293"
+      rpy="3.1416 0 0" />
+    <parent
+      link="base_link" />
+    <child
+      link="U_base_wheel_2_link" />
+    <axis
+      xyz="0 0 -1" />
+    <limit
+      effort="0.323"
+      velocity="10.47" />
+  </joint>
+  <link
+    name="U_wheel_2_link">
+    <inertial>
+      <origin
+        xyz="-0.0015 0 -8.6736E-19"
+        rpy="0 0 0" />
+      <mass
+        value="0.0045951" />
+      <inertia
+        ixx="2.7312E-07"
+        ixy="4.1047E-23"
+        ixz="1.9175E-23"
+        iyy="2.7312E-07"
+        iyz="-7.2378E-23"
+        izz="4.0127E-07" />
+    </inertial>
+    <visual>
+      <origin
+        xyz="0 0 0"
+        rpy="0 0 0" />
+      <geometry>
+        <mesh
+          filename="package://robot_pkg/meshes/U_wheel_2_link.STL" />
+      </geometry>
+      <material
+        name="">
+        <color
+          rgba="1 1 1 1" />
+      </material>
+    </visual>
+    <collision>
+      <origin
+        xyz="0 0 0"
+        rpy="0 0 0" />
+      <geometry>
+        <mesh
+          filename="package://robot_pkg/meshes/U_wheel_2_link.STL" />
+      </geometry>
+    </collision>
+  </link>
+  <joint
+    name="U_wheel_2_joint"
+    type="continuous">
+    <origin
+      xyz="-0.015768 0.00018037 0.016219"
+      rpy="1.5822 -1.5708 0" />
+    <parent
+      link="U_base_wheel_2_link" />
+    <child
+      link="U_wheel_2_link" />
+    <axis
+      xyz="0 0 1" />
+    <limit
+      effort="0.323"
+      velocity="10.47" />
+  </joint>
+  <link
+    name="Support_A_link">
+    <inertial>
+      <origin
+        xyz="0 0 0"
+        rpy="0 0 0" />
+      <mass
+        value="0" />
+      <inertia
+        ixx="0"
+        ixy="0"
+        ixz="0"
+        iyy="0"
+        iyz="0"
+        izz="0" />
+    </inertial>
+    <visual>
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
File: src/robot_pkg/urdf/TTR01.urdf.xacro (robot description, xacro)
@@ -1,3 +1,3 @@
-<?xml version="1.0" encoding="utf-8"?>
+<?xml version="1.0" ?>
 <!-- This URDF was automatically created by SolidWorks to URDF Exporter! Originally created by Stephen Brawner (brawner@gmail.com)
      Commit Version: 1.6.0-4-g7f85cfe  Build Version: 1.6.7995.38578
@@ -592,3 +592,4 @@
       xyz="0 0 0" />
   </joint>
+  <xacro:include filename="gazebo_setup.xacro" /> <!-- -->
 </robot>
