Commit message: new inertial propeties

File: install/robot_pkg/share/robot_pkg/urdf/TTR01.urdf.xacro (robot description, xacro)
@@ -11,12 +11,12 @@
         rpy="0 0 0" />
       <mass
-        value="0.68825" />
-      <inertia
-        ixx="0.00041167"
-        ixy="-1.1043E-10"
-        ixz="-2.4196E-06"
-        iyy="0.00052928"
-        iyz="7.1835E-12"
-        izz="0.00085508" />
+        value="0.7" />
+      <inertia
+        ixx="0.0058"
+        ixy="0"
+        ixz="0"
+        iyy="0.0058"
+        iyz="0"
+        izz="0.0623" />
     </inertial>
     <visual>
@@ -48,15 +48,15 @@
     <inertial>
       <origin
-        xyz="-5.629E-10 5.4357E-10 -0.015886"
-        rpy="0 0 0" />
-      <mass
-        value="0.048724" />
-      <inertia
-        ixx="1.5816E-05"
-        ixy="4.1458E-09"
-        ixz="-1.7893E-13"
-        iyy="1.5814E-05"
-        iyz="1.7858E-13"
-        izz="2.6155E-05" />
+        xyz="-5.629E-10 5.4357E-10 0.0038645"
+        rpy="0 0 0" />
+      <mass
+        value="0.05" />
+      <inertia
+        ixx="0.000056"
+        ixy="0"
+        ixz="0"
+        iyy="0.000056"
+        iyz="0"
+        izz="0.001625" />
     </inertial>
     <visual>
@@ -88,5 +88,5 @@
     type="continuous">
     <origin
-      xyz="0 -0.071 -0.0225"
+      xyz="0 -0.09075 -0.0225"
       rpy="-1.5708 0 0" />
     <parent
@@ -104,15 +104,15 @@
     <inertial>
       <origin
-        xyz="-4.8323E-10 -6.1547E-10 0.015886"
-        rpy="0 0 0" />
-      <mass
-        value="0.048724" />
-      <inertia
-        ixx="1.5817E-05"
-        ixy="-3.7851E-09"
-        ixz="1.5281E-13"
-        iyy="1.5813E-05"
-        iyz="2.0138E-13"
-        izz="2.6155E-05" />
+        xyz="-4.8323E-10 -6.1547E-10 -0.0038645"
+        rpy="0 0 0" />
+      <mass
+        value="0.05" />
+      <inertia
+        ixx="0.000056"
+        ixy="0"
+        ixz="0"
+        iyy="0.000056"
+        iyz="0"
+        izz="0.001625" />
     </inertial>
     <visual>
@@ -144,5 +144,5 @@
     type="continuous">
     <origin
-      xyz="0 0.071 -0.0225"
+      xyz="0 0.09075 -0.0225"
       rpy="-1.5708 0 0" />
     <parent
@@ -160,5 +160,5 @@
     <inertial>
       <origin
-        xyz="0.0041491 -8.4566E-05 0.0063957"
+        xyz="0.0041491 -8.4566E-05 0.0019957"
         rpy="0 0 0" />
       <mass
@@ -200,5 +200,5 @@
     type="continuous">
     <origin
-      xyz="0.057514 0 -0.0234"
+      xyz="0.057514 0 -0.0278"
       rpy="3.1416 0 0" />
     <parent
@@ -216,14 +216,14 @@
     <inertial>
       <origin
-        xyz="-0.0015 0 0"
-        rpy="0 0 0" />
-      <mass
-        value="0.0045951" />
+        xyz="0 -1.3878E-17 6.9389E-18"
+        rpy="0 0 0" />
+      <mass
+        value="0.005" />
       <inertia
         ixx="2.7312E-07"
-        ixy="-2.3056E-23"
-        ixz="-2.2711E-23"
+        ixy="0"
+        ixz="0"
         iyy="2.7312E-07"
-        iyz="-9.4919E-23"
+        iyz="0"
         izz="4.0127E-07" />
     </inertial>
@@ -256,5 +256,5 @@
     type="continuous">
     <origin
-      xyz="0.015768 -0.00018037 0.022119"
+      xyz="0.015768 -0.00018037 0.016219"
       rpy="1.5822 -1.5708 0" />
     <parent
@@ -272,5 +272,5 @@
     <inertial>
       <origin
-        xyz="-0.0041491 8.4566E-05 0.00049565"
+        xyz="-0.0041491 8.4566E-05 0.0019957"
         rpy="0 0 0" />
       <mass
@@ -312,5 +312,5 @@
     type="continuous">
     <origin
-      xyz="-0.057514 0 -0.0293"
+      xyz="-0.057514 0 -0.0278"
       rpy="3.1416 0 0" />
     <parent
@@ -328,5 +328,5 @@
     <inertial>
       <origin
-        xyz="-0.0015 0 -8.6736E-19"
+        xyz="0 0 0"
         rpy="0 0 0" />
       <mass
@@ -334,8 +334,8 @@
       <inertia
         ixx="2.7312E-07"
-        ixy="4.1047E-23"
-        ixz="1.9175E-23"
+        ixy="3.9079E-23"
+        ixz="1.7704E-23"
         iyy="2.7312E-07"
-        iyz="-7.2378E-23"
+        iyz="-6.8863E-23"
         izz="4.0127E-07" />
     </inertial>
@@ -384,15 +384,15 @@
     <inertial>
       <origin
-        xyz="0 0 0"
-        rpy="0 0 0" />
-      <mass
-        value="0" />
-      <inertia
-        ixx="0"
-        ixy="0"
-        ixz="0"
-        iyy="0"
-        iyz="0"
-        izz="0" />
+        xyz="-4.4722E-09 -5.0657E-08 0.00060052"
+        rpy="0 0 0" />
+      <mass
+        value="0.023766" />
+      <inertia
+        ixx="9.5635E-07"
+        ixy="-1.5863E-12"
+        ixz="4.7399E-12"
+        iyy="9.5635E-07"
+        iyz="4.592E-12"
+        izz="9.5992E-08" />
     </inertial>
     <visual>
@@ -407,5 +407,5 @@
         name="">
         <color
-          rgba="1 1 1 1" />
+          rgba="0.75294 0.75294 0.75294 1" />
       </material>
     </visual>
@@ -437,5 +437,5 @@
     <inertial>
       <origin
-        xyz="2.0368E-17 0.00022336 -0.0025145"
+        xyz="7.5901E-18 0.00022336 -1.448E-05"
         rpy="0 0 0" />
       <mass
@@ -443,6 +443,6 @@
       <inertia
         ixx="9.721E-05"
-        ixy="1.83E-21"
-        ixz="3.4946E-22"
+        ixy="9.0124E-22"
+        ixz="1.0137E-22"
         iyy="9.3239E-05"
         iyz="-5.8008E-09"
@@ -477,5 +477,5 @@
     type="fixed">
     <origin
-      xyz="0 0 0.025"
+      xyz="0 0 0.0225"
       rpy="0 0 0" />
     <parent
@@ -530,5 +530,5 @@
     type="fixed">
     <origin
-      xyz="0 0 0.0255"
+      xyz="0 0 0.028"
       rpy="0 0 0" />
     <parent

File: install/robot_pkg/share/robot_pkg/urdf/gazebo_setup.xacro (robot description, xacro)
@@ -1,4 +1,5 @@
 <?xml version="1.0" ?>
 <robot xmlns:xacro="http://www.ros.org/wiki/xacro" name="TTR01">
+    <!-- Define materials for links -->
     <gazebo reference="base_link">
       <material>Gazebo/White</material>
@@ -34,7 +35,7 @@
       <material>Gazebo/White</material>
     </gazebo>
+    <!-- Define plugins -->
     <gazebo>
-        <plugin name="gazebo_ros_joint_state_publisher"
-            filename="libgazebo_ros_joint_state_publisher.so">
+        <plugin name="gazebo_ros_joint_state_publisher" filename="libgazebo_ros_joint_state_publisher.so">
             <update_rate>20</update_rate>
             <joint_name>L_wheel_joint</joint_name>
@@ -47,6 +48,5 @@
     </gazebo>
     <gazebo>
-        <plugin name="gazebo_ros_joint_pose_trajectory"
-            filename="libgazebo_ros_joint_pose_trajectory.so">
+        <plugin name="gazebo_ros_joint_pose_trajectory" filename="libgazebo_ros_joint_pose_trajectory.so">
             <update_rate>2</update_rate>
         </plugin>
