Commit message: new urdf

File: install/robot_pkg/share/robot_pkg/urdf/TTR01.urdf.xacro (robot description, xacro)
@@ -1,595 +1,39 @@
-<?xml version="1.0" ?>
-<!-- This URDF was automatically created by SolidWorks to URDF Exporter! Originally created by Stephen Brawner (brawner@gmail.com)
-     Commit Version: 1.6.0-4-g7f85cfe  Build Version: 1.6.7995.38578
-     For more information, please see http://wiki.ros.org/sw_urdf_exporter -->
-<robot xmlns:xacro="http://www.ros.org/wiki/xacro" name="TTR01">
-  <link
-    name="base_link">
-    <inertial>
-      <origin
-        xyz="0.00041344 3.7856E-10 -0.018281"
-        rpy="0 0 0" />
-      <mass
-        value="0.7" />
-      <inertia
-        ixx="0.0058"
-        ixy="0"
-        ixz="0"
-        iyy="0.0058"
-        iyz="0"
-        izz="0.0623" />
-    </inertial>
-    <visual>
-      <origin
-        xyz="0 0 0"
-        rpy="0 0 0" />
-      <geometry>
-        <mesh
-          filename="package://robot_pkg/meshes/base_link.STL" />
-      </geometry>
-      <material
-        name="">
-        <color
-          rgba="1 1 1 1" />
-      </material>
-    </visual>
-    <collision>
-      <origin
-        xyz="0 0 0"
-        rpy="0 0 0" />
-      <geometry>
-        <mesh
-          filename="package://robot_pkg/meshes/base_link.STL" />
-      </geometry>
-    </collision>
-  </link>
-  <link
-    name="L_wheel_link">
-    <inertial>
-      <origin
-        xyz="-5.629E-10 5.4357E-10 0.0038645"
-        rpy="0 0 0" />
-      <mass
-        value="0.05" />
-      <inertia
-        ixx="0.000056"
-        ixy="0"
-        ixz="0"
-        iyy="0.000056"
-        iyz="0"
-        izz="0.001625" />
-    </inertial>
-    <visual>
-      <origin
-        xyz="0 0 0"
-        rpy="0 0 0" />
-      <geometry>
-        <mesh
-          filename="package://robot_pkg/meshes/L_wheel_link.STL" />
-      </geometry>
-      <material
-        name="">
-        <color
-          rgba="0.75294 0.75294 0.75294 1" />
-      </material>
-    </visual>
-    <collision>
-      <origin
-        xyz="0 0 0"
-        rpy="0 0 0" />
-      <geometry>
-        <mesh
-          filename="package://robot_pkg/meshes/L_wheel_link.STL" />
-      </geometry>
-    </collision>
-  </link>
-  <joint
-    name="L_wheel_joint"
-    type="continuous">
-    <origin
-      xyz="0 -0.09075 -0.0225"
-      rpy="-1.5708 0 0" />
-    <parent
-      link="base_link" />
-    <child
-      link="L_wheel_link" />
-    <axis
-      xyz="0 0 1" />
-    <limit
-      effort="0.323"
-      velocity="10.47" />
-  </joint>
-  <link
-    name="R_wheel_link">
-    <inertial>
-      <origin
-        xyz="-4.8323E-10 -6.1547E-10 -0.0038645"
-        rpy="0 0 0" />
-      <mass
-        value="0.05" />
-      <inertia
-        ixx="0.000056"
-        ixy="0"
-        ixz="0"
-        iyy="0.000056"
-        iyz="0"
-        izz="0.001625" />
-    </inertial>
-    <visual>
-      <origin
-        xyz="0 0 0"
-        rpy="0 0 0" />
-      <geometry>
-        <mesh
-          filename="package://robot_pkg/meshes/R_wheel_link.STL" />
-      </geometry>
-      <material
-        name="">
-        <color
-          rgba="0.75294 0.75294 0.75294 1" />
-      </material>
-    </visual>
-    <collision>
-      <origin
-        xyz="0 0 0"
-        rpy="0 0 0" />
-      <geometry>
-        <mesh
-          filename="package://robot_pkg/meshes/R_wheel_link.STL" />
-      </geometry>
-    </collision>
-  </link>
-  <joint
-    name="R_wheel_joint"
-    type="continuous">
-    <origin
-      xyz="0 0.09075 -0.0225"
-      rpy="-1.5708 0 0" />
-    <parent
-      link="base_link" />
-    <child
-      link="R_wheel_link" />
-    <axis
-      xyz="0 0 1" />
-    <limit
-      effort="0.323"
-      velocity="10.47" />
-  </joint>
-  <link
-    name="U_base_wheel_1_link">
-    <inertial>
-      <origin
-        xyz="0.0041491 -8.4566E-05 0.0019957"
-        rpy="0 0 0" />
-      <mass
-        value="0.009087" />
-      <inertia
-        ixx="5.254E-07"
-        ixy="-4.3301E-10"
-        ixz="-9.4848E-08"
-        iyy="4.8759E-07"
-        iyz="1.0854E-09"
-        izz="7.6419E-07" />
-    </inertial>
-    <visual>
-      <origin
-        xyz="0 0 0"
-        rpy="0 0 0" />
-      <geometry>
-        <mesh
-          filename="package://robot_pkg/meshes/U_base_wheel_1_link.STL" />
-      </geometry>
-      <material
-        name="">
-        <color
-          rgba="0.77647 0.75686 0.73725 1" />
-      </material>
-    </visual>
-    <collision>
-      <origin
-        xyz="0 0 0"
-        rpy="0 0 0" />
-      <geometry>
-        <mesh
-          filename="package://robot_pkg/meshes/U_base_wheel_1_link.STL" />
-      </geometry>
-    </collision>
-  </link>
-  <joint
-    name="U_base_wheel_1_joint"
-    type="continuous">
-    <origin
-      xyz="0.057514 0 -0.0278"
-      rpy="3.1416 0 0" />
-    <parent
-      link="base_link" />
-    <child
-      link="U_base_wheel_1_link" />
-    <axis
-      xyz="0 0 -1" />
-    <limit
-      effort="0.323"
-      velocity="10.47" />
-  </joint>
-  <link
-    name="U_wheel_1_link">
-    <inertial>
-      <origin
-        xyz="0 -1.3878E-17 6.9389E-18"
-        rpy="0 0 0" />
-      <mass
-        value="0.005" />
-      <inertia
-        ixx="2.7312E-07"
-        ixy="0"
-        ixz="0"
-        iyy="2.7312E-07"
-        iyz="0"
-        izz="4.0127E-07" />
-    </inertial>
-    <visual>
-      <origin
-        xyz="0 0 0"
-        rpy="0 0 0" />
-      <geometry>
-        <mesh
-          filename="package://robot_pkg/meshes/U_wheel_1_link.STL" />
-      </geometry>
-      <material
-        name="">
-        <color
-          rgba="1 1 1 1" />
-      </material>
-    </visual>
-    <collision>
-      <origin
-        xyz="0 0 0"
-        rpy="0 0 0" />
-      <geometry>
-        <mesh
-          filename="package://robot_pkg/meshes/U_wheel_1_link.STL" />
-      </geometry>
-    </collision>
-  </link>
-  <joint
-    name="U_wheel_1_joint"
-    type="continuous">
-    <origin
-      xyz="0.015768 -0.00018037 0.016219"
-      rpy="1.5822 -1.5708 0" />
-    <parent
-      link="U_base_wheel_1_link" />
-    <child
-      link="U_wheel_1_link" />
-    <axis
-      xyz="0 0 1" />
-    <limit
-      effort="0.323"
-      velocity="10.47" />
-  </joint>
-  <link
-    name="U_base_wheel_2_link">
-    <inertial>
-      <origin
-        xyz="-0.0041491 8.4566E-05 0.0019957"
-        rpy="0 0 0" />
-      <mass
-        value="0.009087" />
-      <inertia
-        ixx="5.254E-07"
-        ixy="-4.3301E-10"
-        ixz="9.4848E-08"
-        iyy="4.8759E-07"
-        iyz="-1.0854E-09"
-        izz="7.6419E-07" />
-    </inertial>
-    <visual>
-      <origin
-        xyz="0 0 0"
-        rpy="0 0 0" />
-      <geometry>
-        <mesh
-          filename="package://robot_pkg/meshes/U_base_wheel_2_link.STL" />
-      </geometry>
-      <material
-        name="">
-        <color
-          rgba="0.77647 0.75686 0.73725 1" />
-      </material>
-    </visual>
-    <collision>
-      <origin
-        xyz="0 0 0"
-        rpy="0 0 0" />
-      <geometry>
-        <mesh
-          filename="package://robot_pkg/meshes/U_base_wheel_2_link.STL" />
-      </geometry>
-    </collision>
-  </link>
-  <joint
-    name="U_base_wheel_2_joint"
-    type="continuous">
-    <origin
-      xyz="-0.057514 0 -0.0278"
-      rpy="3.1416 0 0" />
-    <parent
-      link="base_link" />
-    <child
-      link="U_base_wheel_2_link" />
-    <axis
-      xyz="0 0 -1" />
-    <limit
-      effort="0.323"
-      velocity="10.47" />
-  </joint>
-  <link
-    name="U_wheel_2_link">
-    <inertial>
-      <origin
-        xyz="0 0 0"
-        rpy="0 0 0" />
-      <mass
-        value="0.0045951" />
-      <inertia
-        ixx="2.7312E-07"
-        ixy="3.9079E-23"
-        ixz="1.7704E-23"
-        iyy="2.7312E-07"
-        iyz="-6.8863E-23"
-        izz="4.0127E-07" />
-    </inertial>
-    <visual>
-      <origin
-        xyz="0 0 0"
-        rpy="0 0 0" />
-      <geometry>
-        <mesh
-          filename="package://robot_pkg/meshes/U_wheel_2_link.STL" />
-      </geometry>
-      <material
-        name="">
-        <color
-          rgba="1 1 1 1" />
-      </material>
-    </visual>
-    <collision>
-      <origin
-        xyz="0 0 0"
-        rpy="0 0 0" />
-      <geometry>
-        <mesh
-          filename="package://robot_pkg/meshes/U_wheel_2_link.STL" />
-      </geometry>
-    </collision>
-  </link>
-  <joint
-    name="U_wheel_2_joint"
-    type="continuous">
-    <origin
-      xyz="-0.015768 0.00018037 0.016219"
-      rpy="1.5822 -1.5708 0" />
-    <parent
-      link="U_base_wheel_2_link" />
-    <child
-      link="U_wheel_2_link" />
-    <axis
-      xyz="0 0 1" />
-    <limit
-      effort="0.323"
-      velocity="10.47" />
-  </joint>
-  <link
-    name="Support_A_link">
-    <inertial>
-      <origin
-        xyz="-4.4722E-09 -5.0657E-08 0.00060052"
-        rpy="0 0 0" />
-      <mass
-        value="0.023766" />
-      <inertia
-        ixx="9.5635E-07"
-        ixy="-1.5863E-12"
-        ixz="4.7399E-12"
-        iyy="9.5635E-07"
-        iyz="4.592E-12"
-        izz="9.5992E-08" />
-    </inertial>
-    <visual>
-      <origin
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
File: install/robot_pkg/share/robot_pkg/urdf/gazebo_setup.xacro (robot description, xacro)
@@ -1,3 +1,3 @@
-<?xml version="1.0" ?>
+<?xml version="1.0"?>
 <robot xmlns:xacro="http://www.ros.org/wiki/xacro" name="TTR01">
     <!-- Define materials for links -->

File: src/robot_pkg/urdf/TTR01.urdf.xacro (robot description, xacro)
@@ -1,595 +1,40 @@
-<?xml version="1.0" ?>
-<!-- This URDF was automatically created by SolidWorks to URDF Exporter! Originally created by Stephen Brawner (brawner@gmail.com)
-     Commit Version: 1.6.0-4-g7f85cfe  Build Version: 1.6.7995.38578
-     For more information, please see http://wiki.ros.org/sw_urdf_exporter -->
-<robot xmlns:xacro="http://www.ros.org/wiki/xacro" name="TTR01">
-  <link
-    name="base_link">
-    <inertial>
-      <origin
-        xyz="0.00041344 3.7856E-10 -0.018281"
-        rpy="0 0 0" />
-      <mass
-        value="0.7" />
-      <inertia
-        ixx="0.0058"
-        ixy="0"
-        ixz="0"
-        iyy="0.0058"
-        iyz="0"
-        izz="0.0623" />
-    </inertial>
-    <visual>
-      <origin
-        xyz="0 0 0"
-        rpy="0 0 0" />
-      <geometry>
-        <mesh
-          filename="package://robot_pkg/meshes/base_link.STL" />
-      </geometry>
-      <material
-        name="">
-        <color
-          rgba="1 1 1 1" />
-      </material>
-    </visual>
-    <collision>
-      <origin
-        xyz="0 0 0"
-        rpy="0 0 0" />
-      <geometry>
-        <mesh
-          filename="package://robot_pkg/meshes/base_link.STL" />
-      </geometry>
-    </collision>
-  </link>
-  <link
-    name="L_wheel_link">
-    <inertial>
-      <origin
-        xyz="-5.629E-10 5.4357E-10 0.0038645"
-        rpy="0 0 0" />
-      <mass
-        value="0.05" />
-      <inertia
-        ixx="0.000056"
-        ixy="0"
-        ixz="0"
-        iyy="0.000056"
-        iyz="0"
-        izz="0.001625" />
-    </inertial>
-    <visual>
-      <origin
-        xyz="0 0 0"
-        rpy="0 0 0" />
-      <geometry>
-        <mesh
-          filename="package://robot_pkg/meshes/L_wheel_link.STL" />
-      </geometry>
-      <material
-        name="">
-        <color
-          rgba="0.75294 0.75294 0.75294 1" />
-      </material>
-    </visual>
-    <collision>
-      <origin
-        xyz="0 0 0"
-        rpy="0 0 0" />
-      <geometry>
-        <mesh
-          filename="package://robot_pkg/meshes/L_wheel_link.STL" />
-      </geometry>
-    </collision>
-  </link>
-  <joint
-    name="L_wheel_joint"
-    type="continuous">
-    <origin
-      xyz="0 -0.09075 -0.0225"
-      rpy="-1.5708 0 0" />
-    <parent
-      link="base_link" />
-    <child
-      link="L_wheel_link" />
-    <axis
-      xyz="0 0 1" />
-    <limit
-      effort="0.323"
-      velocity="10.47" />
-  </joint>
-  <link
-    name="R_wheel_link">
-    <inertial>
-      <origin
-        xyz="-4.8323E-10 -6.1547E-10 -0.0038645"
-        rpy="0 0 0" />
-      <mass
-        value="0.05" />
-      <inertia
-        ixx="0.000056"
-        ixy="0"
-        ixz="0"
-        iyy="0.000056"
-        iyz="0"
-        izz="0.001625" />
-    </inertial>
-    <visual>
-      <origin
-        xyz="0 0 0"
-        rpy="0 0 0" />
-      <geometry>
-        <mesh
-          filename="package://robot_pkg/meshes/R_wheel_link.STL" />
-      </geometry>
-      <material
-        name="">
-        <color
-          rgba="0.75294 0.75294 0.75294 1" />
-      </material>
-    </visual>
-    <collision>
-      <origin
-        xyz="0 0 0"
-        rpy="0 0 0" />
-      <geometry>
-        <mesh
-          filename="package://robot_pkg/meshes/R_wheel_link.STL" />
-      </geometry>
-    </collision>
-  </link>
-  <joint
-    name="R_wheel_joint"
-    type="continuous">
-    <origin
-      xyz="0 0.09075 -0.0225"
-      rpy="-1.5708 0 0" />
-    <parent
-      link="base_link" />
-    <child
-      link="R_wheel_link" />
-    <axis
-      xyz="0 0 1" />
-    <limit
-      effort="0.323"
-      velocity="10.47" />
-  </joint>
-  <link
-    name="U_base_wheel_1_link">
-    <inertial>
-      <origin
-        xyz="0.0041491 -8.4566E-05 0.0019957"
-        rpy="0 0 0" />
-      <mass
-        value="0.009087" />
-      <inertia
-        ixx="5.254E-07"
-        ixy="-4.3301E-10"
-        ixz="-9.4848E-08"
-        iyy="4.8759E-07"
-        iyz="1.0854E-09"
-        izz="7.6419E-07" />
-    </inertial>
-    <visual>
-      <origin
-        xyz="0 0 0"
-        rpy="0 0 0" />
-      <geometry>
-        <mesh
-          filename="package://robot_pkg/meshes/U_base_wheel_1_link.STL" />
-      </geometry>
-      <material
-        name="">
-        <color
-          rgba="0.77647 0.75686 0.73725 1" />
-      </material>
-    </visual>
-    <collision>
-      <origin
-        xyz="0 0 0"
-        rpy="0 0 0" />
-      <geometry>
-        <mesh
-          filename="package://robot_pkg/meshes/U_base_wheel_1_link.STL" />
-      </geometry>
-    </collision>
-  </link>
-  <joint
-    name="U_base_wheel_1_joint"
-    type="continuous">
-    <origin
-      xyz="0.057514 0 -0.0278"
-      rpy="3.1416 0 0" />
-    <parent
-      link="base_link" />
-    <child
-      link="U_base_wheel_1_link" />
-    <axis
-      xyz="0 0 -1" />
-    <limit
-      effort="0.323"
-      velocity="10.47" />
-  </joint>
-  <link
-    name="U_wheel_1_link">
-    <inertial>
-      <origin
-        xyz="0 -1.3878E-17 6.9389E-18"
-        rpy="0 0 0" />
-      <mass
-        value="0.005" />
-      <inertia
-        ixx="2.7312E-07"
-        ixy="0"
-        ixz="0"
-        iyy="2.7312E-07"
-        iyz="0"
-        izz="4.0127E-07" />
-    </inertial>
-    <visual>
-      <origin
-        xyz="0 0 0"
-        rpy="0 0 0" />
-      <geometry>
-        <mesh
-          filename="package://robot_pkg/meshes/U_wheel_1_link.STL" />
-      </geometry>
-      <material
-        name="">
-        <color
-          rgba="1 1 1 1" />
-      </material>
-    </visual>
-    <collision>
-      <origin
-        xyz="0 0 0"
-        rpy="0 0 0" />
-      <geometry>
-        <mesh
-          filename="package://robot_pkg/meshes/U_wheel_1_link.STL" />
-      </geometry>
-    </collision>
-  </link>
-  <joint
-    name="U_wheel_1_joint"
-    type="continuous">
-    <origin
-      xyz="0.015768 -0.00018037 0.016219"
-      rpy="1.5822 -1.5708 0" />
-    <parent
-      link="U_base_wheel_1_link" />
-    <child
-      link="U_wheel_1_link" />
-    <axis
-      xyz="0 0 1" />
-    <limit
-      effort="0.323"
-      velocity="10.47" />
-  </joint>
-  <link
-    name="U_base_wheel_2_link">
-    <inertial>
-      <origin
-        xyz="-0.0041491 8.4566E-05 0.0019957"
-        rpy="0 0 0" />
-      <mass
-        value="0.009087" />
-      <inertia
-        ixx="5.254E-07"
-        ixy="-4.3301E-10"
-        ixz="9.4848E-08"
-        iyy="4.8759E-07"
-        iyz="-1.0854E-09"
-        izz="7.6419E-07" />
-    </inertial>
-    <visual>
-      <origin
-        xyz="0 0 0"
-        rpy="0 0 0" />
-      <geometry>
-        <mesh
-          filename="package://robot_pkg/meshes/U_base_wheel_2_link.STL" />
-      </geometry>
-      <material
-        name="">
-        <color
-          rgba="0.77647 0.75686 0.73725 1" />
-      </material>
-    </visual>
-    <collision>
-      <origin
-        xyz="0 0 0"
-        rpy="0 0 0" />
-      <geometry>
-        <mesh
-          filename="package://robot_pkg/meshes/U_base_wheel_2_link.STL" />
-      </geometry>
-    </collision>
-  </link>
-  <joint
-    name="U_base_wheel_2_joint"
-    type="continuous">
-    <origin
-      xyz="-0.057514 0 -0.0278"
-      rpy="3.1416 0 0" />
-    <parent
-      link="base_link" />
-    <child
-      link="U_base_wheel_2_link" />
-    <axis
-      xyz="0 0 -1" />
-    <limit
-      effort="0.323"
-      velocity="10.47" />
-  </joint>
-  <link
-    name="U_wheel_2_link">
-    <inertial>
-      <origin
-        xyz="0 0 0"
-        rpy="0 0 0" />
-      <mass
-        value="0.0045951" />
-      <inertia
-        ixx="2.7312E-07"
-        ixy="3.9079E-23"
-        ixz="1.7704E-23"
-        iyy="2.7312E-07"
-        iyz="-6.8863E-23"
-        izz="4.0127E-07" />
-    </inertial>
-    <visual>
-      <origin
-        xyz="0 0 0"
-        rpy="0 0 0" />
-      <geometry>
-        <mesh
-          filename="package://robot_pkg/meshes/U_wheel_2_link.STL" />
-      </geometry>
-      <material
-        name="">
-        <color
-          rgba="1 1 1 1" />
-      </material>
-    </visual>
-    <collision>
-      <origin
-        xyz="0 0 0"
-        rpy="0 0 0" />
-      <geometry>
-        <mesh
-          filename="package://robot_pkg/meshes/U_wheel_2_link.STL" />
-      </geometry>
-    </collision>
-  </link>
-  <joint
-    name="U_wheel_2_joint"
-    type="continuous">
-    <origin
-      xyz="-0.015768 0.00018037 0.016219"
-      rpy="1.5822 -1.5708 0" />
-    <parent
-      link="U_base_wheel_2_link" />
-    <child
-      link="U_wheel_2_link" />
-    <axis
-      xyz="0 0 1" />
-    <limit
-      effort="0.323"
-      velocity="10.47" />
-  </joint>
-  <link
-    name="Support_A_link">
-    <inertial>
-      <origin
-        xyz="-4.4722E-09 -5.0657E-08 0.00060052"
-        rpy="0 0 0" />
-      <mass
-        value="0.023766" />
-      <inertia
-        ixx="9.5635E-07"
-        ixy="-1.5863E-12"
-        ixz="4.7399E-12"
-        iyy="9.5635E-07"
-        iyz="4.592E-12"
-        izz="9.5992E-08" />
-    </inertial>
-    <visual>
-      <origin
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