Commit message: urdf_v1

File: install/robot_pkg/share/robot_pkg/urdf/TTR01.urdf.xacro (robot description, xacro)
@@ -3,16 +3,16 @@
     <!--world frame-->
     <xacro:include filename="parameters.xacro"/>
-    <link name="World"> </link>
-    <joint name="World_joint" type="fixed">
-        <origin xyz="0 0 0" rpy="0 0 0"/>
-        <parent link="World"/>
-        <child link="base_link"/>
+    <link name="base_link"> </link>
+    <!--base frame-->
+    <joint name="B_base_joint" type="fixed">
+        <origin xyz="0 0 0.05606" rpy="0 0 0"/>
+        <parent link="base_link"/>
+        <child link="B_base_link"/>
     </joint>
-    <!--base frame-->
     <xacro:property name="B_base_length" value="0.005"/>
-    <xacro:property name="B_base_radius" value="0.178"/>
-    <link name="base_link">
+    <xacro:property name="B_base_radius" value="0.085"/>
+    <link name="B_base_link">
         <visual>
-            <origin xyz="0 0 ${B_base_length/2}" rpy="0 0 0"/>
+            <origin xyz="0 0 0" rpy="0 0 0"/>
             <geometry>
                 <!--<mesh filename="package://robot_pkg/meshes/base_link.STL" />-->
@@ -22,18 +22,68 @@
         </visual>
         <collision>
-            <origin xyz="0 0 ${B_base_length/2}" rpy="0 0 0"/>
+            <origin xyz="0 0 0" rpy="0 0 0"/>
             <geometry>
+                <!--<mesh filename="package://robot_pkg/meshes/base_link.STL" />-->
                 <cylinder length="${B_base_length}" radius="${B_base_radius}"/>
             </geometry>
         </collision>
         <xacro:inertial_cylinder mass="0.9" length="${B_base_length}" radius="${B_base_radius}">
-            <origin xyz="0 0 0.034" rpy="0 0 0"/>
+            <origin xyz="0 0 0.05606" rpy="0 0 0"/>
         </xacro:inertial_cylinder>
     </link>
-    <joint name="base_joint" type="fixed">
-        <origin xyz="0 0 0.034" rpy="0 0 0"/>
-        <parent link="World"/>
-        <child link="base_link"/>
+    <!--L_wheel_frame-->
+    <joint name="L_wheel_joint" type="continuous">
+        <origin xyz="0 -0.0986 -0.0225" rpy="${-pi/2} ${-pi/2} ${pi}"/>
+        <parent link="B_base_link"/>
+        <child link="L_wheel_link"/>
+        <axis xyz="0 0 1"/>
+        <limit effort="0.323" velocity="10.47" />
     </joint>
+    <xacro:property name="wheel_thickness" value="0.027"/>
+    <xacro:property name="wheel_radius" value="0.0325"/>
+    <link name="L_wheel_link">
+        <visual>
+            <origin xyz="0 0 0" rpy="0 0 0"/>
+            <geometry>
+                <cylinder length="${wheel_thickness}" radius="${wheel_radius}"/>
+            </geometry>
+            <material name="black"/>
+        </visual>
+        <collision>
+            <origin xyz="0 0 0" rpy="0 0 0"/>
+            <geometry>
+                <cylinder length="${wheel_thickness}" radius="${wheel_radius}"/>
+            </geometry>
+        </collision>
+        <xacro:inertial_cylinder mass="0.05" length="${wheel_thickness}" radius="${wheel_radius}">
+            <origin xyz="0 -0.0986 -0.023" rpy="${-pi/2} ${-pi/2} ${pi}"/>
+        </xacro:inertial_cylinder>
+    </link>
+    <!--R_wheel_frame-->
+    <joint name="R_wheel_joint" type="continuous">
+        <origin xyz="0 0.0986 -0.0225" rpy="${-pi/2} ${pi/2} 0"/>
+        <parent link="B_base_link"/>
+        <child link="R_wheel_link"/>
+        <axis xyz="0 0 -1"/>
+        <limit effort="0.323" velocity="10.47" />
+    </joint>
+    <link name="R_wheel_link">
+        <visual>
+            <origin xyz="0 0 0" rpy="0 0 0"/>
+            <geometry>
+                <cylinder length="${wheel_thickness}" radius="${wheel_radius}"/>
+            </geometry>
+            <material name="black"/>
+        </visual>
+        <collision>
+            <origin xyz="0 0 0" rpy="0 0 0"/>
+            <geometry>
+                <cylinder length="${wheel_thickness}" radius="${wheel_radius}"/>
+            </geometry>
+        </collision>
+        <xacro:inertial_cylinder mass="0.05" length="${wheel_thickness}" radius="${wheel_radius}">
+            <origin xyz="0 0.0986 -0.0225" rpy="${-pi/2} ${pi/2} 0"/>
+        </xacro:inertial_cylinder>
+    </link>
     <xacro:include filename="gazebo_setup.xacro"/>
 </robot>

File: install/robot_pkg/share/robot_pkg/urdf/gazebo_setup.xacro (robot description, xacro)
@@ -6,5 +6,5 @@
     </gazebo>
     <gazebo reference="L_wheel_link">
-      <material>Gazebo/White</material>
+      <material>Gazebo/Black</material>
     </gazebo>
     <gazebo reference="R_wheel_link">
@@ -23,15 +23,29 @@
       <material>Gazebo/White</material>
     </gazebo>
-    <gazebo reference="Support_A_link">
+    <gazebo reference="Support_link">
       <material>Gazebo/Yellow</material>
     </gazebo>
-    <gazebo reference="M_base_link">
-      <material>Gazebo/White</material>
+    <!-- Define friction for wheels -->
+    <gazebo reference="L_wheel_link">
+        <material>Gazebo/Black</material>
+        <surface>
+            <friction>
+                <ode>
+                    <mu>1.0</mu> <!-- Fricción estática -->
+                    <mu2>0.8</mu2> <!-- Fricción dinámica -->
+                </ode>
+            </friction>
+        </surface>
     </gazebo>
-    <gazebo reference="Support_B_link">
-      <material>Gazebo/Yellow</material>
-    </gazebo>
-    <gazebo reference="T_base_link">
-      <material>Gazebo/White</material>
+    <gazebo reference="R_wheel_link">
+        <material>Gazebo/Black</material>
+        <surface>
+            <friction>
+                <ode>
+                    <mu>1.0</mu>
+                    <mu2>0.8</mu2>
+                </ode>
+            </friction>
+        </surface>
     </gazebo>
     <!-- Define plugins -->
@@ -41,8 +55,8 @@
             <joint_name>L_wheel_joint</joint_name>
             <joint_name>R_wheel_joint</joint_name>
-            <joint_name>U_base_wheel_1_joint</joint_name>
+            <!--<joint_name>U_base_wheel_1_joint</joint_name>
             <joint_name>U_wheel_1_joint</joint_name>
             <joint_name>U_base_wheel_2_joint</joint_name>
-            <joint_name>U_wheel_2_joint</joint_name>
+            <joint_name>U_wheel_2_joint</joint_name>-->
         </plugin>
     </gazebo>
@@ -52,3 +66,14 @@
         </plugin>
     </gazebo>
+    <!-- Differential drive plugin for moving the robot -->
+    <gazebo>
+        <plugin name="diff_drive_controller" filename="libgazebo_ros_diff_drive.so">
+            <update_rate>50</update_rate>
+            <left_joint>L_wheel_joint</left_joint>
+            <right_joint>R_wheel_joint</right_joint>
+            <wheel_separation>0.2115</wheel_separation> <!-- Adjust according to your robot -->
+            <wheel_diameter>0.065</wheel_diameter> <!-- Adjust according to your wheels -->
+            <robot_base_frame>base_link</robot_base_frame>
+        </plugin>
+    </gazebo>
 </robot>

File: src/robot_pkg/urdf/TTR01.urdf.xacro (robot description, xacro)
@@ -3,16 +3,16 @@
     <!--world frame-->
     <xacro:include filename="parameters.xacro"/>
-    <link name="World"> </link>
-    <joint name="World_joint" type="fixed">
-        <origin xyz="0 0 0" rpy="0 0 0"/>
-        <parent link="World"/>
-        <child link="base_link"/>
+    <link name="base_link"> </link>
+    <!--base frame-->
+    <joint name="B_base_joint" type="fixed">
+        <origin xyz="0 0 0.05606" rpy="0 0 0"/>
+        <parent link="base_link"/>
+        <child link="B_base_link"/>
     </joint>
-    <!--base frame-->
     <xacro:property name="B_base_length" value="0.005"/>
-    <xacro:property name="B_base_radius" value="0.178"/>
-    <link name="base_link">
+    <xacro:property name="B_base_radius" value="0.085"/>
+    <link name="B_base_link">
         <visual>
-            <origin xyz="0 0 ${B_base_length/2}" rpy="0 0 0"/>
+            <origin xyz="0 0 0" rpy="0 0 0"/>
             <geometry>
                 <!--<mesh filename="package://robot_pkg/meshes/base_link.STL" />-->
@@ -22,5 +22,5 @@
         </visual>
         <collision>
-            <origin xyz="0 0 ${B_base_length/2}" rpy="0 0 0"/>
+            <origin xyz="0 0 0" rpy="0 0 0"/>
             <geometry>
                 <!--<mesh filename="package://robot_pkg/meshes/base_link.STL" />-->
@@ -29,12 +29,61 @@
         </collision>
         <xacro:inertial_cylinder mass="0.9" length="${B_base_length}" radius="${B_base_radius}">
-            <origin xyz="0 0 0.034" rpy="0 0 0"/>
+            <origin xyz="0 0 0.05606" rpy="0 0 0"/>
         </xacro:inertial_cylinder>
     </link>
-    <joint name="base_joint" type="fixed">
-        <origin xyz="0 0 0.034" rpy="0 0 0"/>
-        <parent link="World"/>
-        <child link="base_link"/>
+    <!--L_wheel_frame-->
+    <joint name="L_wheel_joint" type="continuous">
+        <origin xyz="0 -0.0986 -0.0225" rpy="${-pi/2} ${-pi/2} ${pi}"/>
+        <parent link="B_base_link"/>
+        <child link="L_wheel_link"/>
+        <axis xyz="0 0 1"/>
+        <limit effort="0.323" velocity="10.47" />
     </joint>
+    <xacro:property name="wheel_thickness" value="0.027"/>
+    <xacro:property name="wheel_radius" value="0.0325"/>
+    <link name="L_wheel_link">
+        <visual>
+            <origin xyz="0 0 0" rpy="0 0 0"/>
+            <geometry>
+                <cylinder length="${wheel_thickness}" radius="${wheel_radius}"/>
+            </geometry>
+            <material name="black"/>
+        </visual>
+        <collision>
+            <origin xyz="0 0 0" rpy="0 0 0"/>
+            <geometry>
+                <cylinder length="${wheel_thickness}" radius="${wheel_radius}"/>
+            </geometry>
+        </collision>
+        <xacro:inertial_cylinder mass="0.05" length="${wheel_thickness}" radius="${wheel_radius}">
+            <origin xyz="0 -0.0986 -0.023" rpy="${-pi/2} ${-pi/2} ${pi}"/>
+        </xacro:inertial_cylinder>
+    </link>
+    <!--R_wheel_frame-->
+    <joint name="R_wheel_joint" type="continuous">
+        <origin xyz="0 0.0986 -0.0225" rpy="${-pi/2} ${pi/2} 0"/>
+        <parent link="B_base_link"/>
+        <child link="R_wheel_link"/>
+        <axis xyz="0 0 -1"/>
+        <limit effort="0.323" velocity="10.47" />
+    </joint>
+    <link name="R_wheel_link">
+        <visual>
+            <origin xyz="0 0 0" rpy="0 0 0"/>
+            <geometry>
+                <cylinder length="${wheel_thickness}" radius="${wheel_radius}"/>
+            </geometry>
+            <material name="black"/>
+        </visual>
+        <collision>
+            <origin xyz="0 0 0" rpy="0 0 0"/>
+            <geometry>
+                <cylinder length="${wheel_thickness}" radius="${wheel_radius}"/>
+            </geometry>
+        </collision>
+        <xacro:inertial_cylinder mass="0.05" length="${wheel_thickness}" radius="${wheel_radius}">
+            <origin xyz="0 0.0986 -0.0225" rpy="${-pi/2} ${pi/2} 0"/>
+        </xacro:inertial_cylinder>
+    </link>
     <xacro:include filename="gazebo_setup.xacro"/>
 </robot>

Commit message: new urdf 2

File: install/robot_pkg/share/robot_pkg/urdf/TTR01.urdf.xacro (robot description, xacro)
@@ -1,8 +1,8 @@
 <?xml version="1.0"?>
 <robot xmlns:xacro="http://www.ros.org/wiki/xacro"  name="TTR01">
-    <!--world frame-->
-    <xacro:include filename="parameters.xacro"/>
+    <!--base/world frame-->
+    <xacro:include filename="robot_parameters.xacro"/>
     <link name="base_link"> </link>
-    <!--base frame-->
+    <!--Bottom base frame-->
     <joint name="B_base_joint" type="fixed">
         <origin xyz="0 0 0.05606" rpy="0 0 0"/>
@@ -11,8 +11,8 @@
     </joint>
     <xacro:property name="B_base_length" value="0.005"/>
-    <xacro:property name="B_base_radius" value="0.085"/>
+    <xacro:property name="B_base_radius" value="0.089"/>
     <link name="B_base_link">
         <visual>
-            <origin xyz="0 0 0" rpy="0 0 0"/>
+            <origin xyz="0 0 -${B_base_length/2}" rpy="0 0 0"/>
             <geometry>
                 <!--<mesh filename="package://robot_pkg/meshes/base_link.STL" />-->
@@ -22,5 +22,5 @@
         </visual>
         <collision>
-            <origin xyz="0 0 0" rpy="0 0 0"/>
+            <origin xyz="0 0 -${B_base_length/2}" rpy="0 0 0"/>
             <geometry>
                 <!--<mesh filename="package://robot_pkg/meshes/base_link.STL" />-->
@@ -32,7 +32,7 @@
         </xacro:inertial_cylinder>
     </link>
-    <!--L_wheel_frame-->
+    <!--Left wheel frame-->
     <joint name="L_wheel_joint" type="continuous">
-        <origin xyz="0 -0.0986 -0.0225" rpy="${-pi/2} ${-pi/2} ${pi}"/>
+        <origin xyz="0 -0.10575 -0.0225" rpy="${-pi/2} ${-pi/2} ${pi}"/>
         <parent link="B_base_link"/>
         <child link="L_wheel_link"/>
@@ -57,10 +57,10 @@
         </collision>
         <xacro:inertial_cylinder mass="0.05" length="${wheel_thickness}" radius="${wheel_radius}">
-            <origin xyz="0 -0.0986 -0.023" rpy="${-pi/2} ${-pi/2} ${pi}"/>
+            <origin xyz="0 -0.10575 -0.023" rpy="${-pi/2} ${-pi/2} ${pi}"/>
         </xacro:inertial_cylinder>
     </link>
-    <!--R_wheel_frame-->
+    <!--Right wheel frame-->
     <joint name="R_wheel_joint" type="continuous">
-        <origin xyz="0 0.0986 -0.0225" rpy="${-pi/2} ${pi/2} 0"/>
+        <origin xyz="0 0.10575 -0.0225" rpy="${-pi/2} ${pi/2} 0"/>
         <parent link="B_base_link"/>
         <child link="R_wheel_link"/>
@@ -83,5 +83,114 @@
         </collision>
         <xacro:inertial_cylinder mass="0.05" length="${wheel_thickness}" radius="${wheel_radius}">
-            <origin xyz="0 0.0986 -0.0225" rpy="${-pi/2} ${pi/2} 0"/>
+            <origin xyz="0 0.10575 -0.0225" rpy="${-pi/2} ${pi/2} 0"/>
+        </xacro:inertial_cylinder>
+    </link>
+    <!--Caster wheel base 1-->
+    <joint name="U_base_wheel_1_joint" type="continuous">
+        <origin xyz="0.05751 0 -0.0278" rpy="${pi} 0 0"/>
+        <parent link="B_base_link"/>
+        <child link="U_base_wheel_1_link"/>
+        <axis xyz="0 0 -1"/>
+        <limit effort="0.323" velocity="10.47" />
+    </joint>
+    <xacro:property name="U_base_box_X" value="0.028"/>
+    <xacro:property name="U_base_box_Y" value="0.032"/>
+    <xacro:property name="U_base_box_Z" value="0.04402"/>
+    <link name="U_base_wheel_1_link">
+        <visual>
+            <origin xyz="0 0 0" rpy="0 0 0"/>
+            <geometry>
+                <box size="${U_base_box_X} ${U_base_box_Y} ${U_base_box_Z}"/>
+            </geometry>
+            <material name="light_gray"/>
+        </visual>
+        <collision>
+            <origin xyz="0 0 0" rpy="0 0 0"/>
+            <geometry>
+                <box size="${U_base_box_X} ${U_base_box_Y} ${U_base_box_Z}"/>
+            </geometry>
+        </collision>
+        <xacro:inertial_box mass="0.0125" x="${U_base_box_X}" y="${U_base_box_Y}" z="${U_base_box_Z}">
+            <origin xyz="0.05751 0 -0.0278" rpy="${pi} 0 0"/>
+        </xacro:inertial_box>
+    </link>
+    <!--Caster wheel 1-->
+    <joint name="U_wheel_1_joint" type="continuous">
+        <origin xyz="0.01577 0 0.01622" rpy="${pi/2} 0 0"/>
+        <parent link="U_base_wheel_1_link"/>
+        <child link="U_wheel_1_link"/>
+        <axis xyz="0 0 1"/>
+        <limit effort="0.323" velocity="10.47" />
+    </joint>
+    <xacro:property name="U_wheel_thickness" value="0.0144"/>
+    <xacro:property name="U_wheel_radius" value="0.0115"/>
+    <link name="U_wheel_1_link">
+        <visual>
+            <origin xyz="0 0 0" rpy="0 0 0"/>
+            <geometry>
+                <cylinder radius="${U_wheel_radius}" length="${U_wheel_thickness}"/>
+            </geometry>
+            <material name="white"/>
+        </visual>
+        <collision>
+            <origin xyz="0 0 0" rpy="0 0 0"/>
+            <geometry>
+                <cylinder radius="${U_wheel_radius}" length="${U_wheel_thickness}"/>
+            </geometry>
+        </collision>
+        <xacro:inertial_cylinder mass="0.005" length="${U_wheel_thickness}" radius="${U_wheel_radius}">
+            <origin xyz="0.01577 0 0.01622" rpy="${pi/2} 0 ${pi/2}"/>
+        </xacro:inertial_cylinder>
+    </link>
+    <!--Caster wheel base 2-->
+    <joint name="U_base_wheel_2_joint" type="continuous">
+        <origin xyz="-0.05751 0 -0.0278" rpy="${pi} 0 ${pi}"/>
+        <parent link="B_base_link"/>
+        <child link="U_base_wheel_2_link"/>
+        <axis xyz="0 0 -1"/>
+        <limit effort="0.323" velocity="10.47" />
+    </joint>
+    <link name="U_base_wheel_2_link">
+        <visual>
+            <origin xyz="0 0 0" rpy="0 0 0"/>
+            <geometry>
+                <box size="${U_base_box_X} ${U_base_box_Y} ${U_base_box_Z}"/>
+            </geometry>
+            <material name="light_gray"/>
+        </visual>
+        <collision>
+            <origin xyz="0 0 0" rpy="0 0 0"/>
+            <geometry>
+                <box size="${U_base_box_X} ${U_base_box_Y} ${U_base_box_Z}"/>
+            </geometry>
+        </collision>
+        <xacro:inertial_box mass="0.0125" x="${U_base_box_X}" y="${U_base_box_Y}" z="${U_base_box_Z}">
+            <origin xyz="-0.05751 0 -0.0278" rpy="${pi} 0 0"/>
+        </xacro:inertial_box>
+    </link>
+    <!--Caster wheel 2-->
+    <joint name="U_wheel_2_joint" type="continuous">
+        <origin xyz="0.01577 0 0.01622" rpy="${pi/2} 0 0"/>
+        <parent link="U_base_wheel_2_link"/>
+        <child link="U_wheel_2_link"/>
+        <axis xyz="0 0 1"/>
+        <limit effort="0.323" velocity="10.47" />
+    </joint>
+    <link name="U_wheel_2_link">
+        <visual>
+            <origin xyz="0 0 0" rpy="0 0 0"/>
+            <geometry>
+                <cylinder radius="${U_wheel_radius}" length="${U_wheel_thickness}"/>
+            </geometry>
+            <material name="white"/>
+        </visual>
+        <collision>
+            <origin xyz="0 0 0" rpy="0 0 0"/>
+            <geometry>
+                <cylinder radius="${U_wheel_radius}" length="${U_wheel_thickness}"/>
+            </geometry>
+        </collision>
+        <xacro:inertial_cylinder mass="0.005" length="${U_wheel_thickness}" radius="${U_wheel_radius}">
+            <origin xyz="0.01577 0 0.01622" rpy="${pi/2} 0 ${pi/2}"/>
         </xacro:inertial_cylinder>
     </link>

File: install/robot_pkg/share/robot_pkg/urdf/gazebo_setup.xacro (robot description, xacro)
@@ -55,8 +55,8 @@
             <joint_name>L_wheel_joint</joint_name>
             <joint_name>R_wheel_joint</joint_name>
-            <!--<joint_name>U_base_wheel_1_joint</joint_name>
+            <joint_name>U_base_wheel_1_joint</joint_name>
             <joint_name>U_wheel_1_joint</joint_name>
             <joint_name>U_base_wheel_2_joint</joint_name>
-            <joint_name>U_wheel_2_joint</joint_name>-->
+            <joint_name>U_wheel_2_joint</joint_name>
         </plugin>
     </gazebo>
