Commit message: almost final urdf

File: install/robot_pkg/share/robot_pkg/urdf/TTR01.urdf.xacro (robot description, xacro)
@@ -29,5 +29,5 @@
         </collision>
         <xacro:inertial_cylinder mass="0.9" length="${B_base_length}" radius="${B_base_radius}">
-            <origin xyz="0 0 0.05606" rpy="0 0 0"/>
+            <origin xyz="0 0 -${B_base_length/2}" rpy="0 0 0"/>
         </xacro:inertial_cylinder>
     </link>
@@ -57,5 +57,5 @@
         </collision>
         <xacro:inertial_cylinder mass="0.05" length="${wheel_thickness}" radius="${wheel_radius}">
-            <origin xyz="0 -0.10575 -0.023" rpy="${-pi/2} ${-pi/2} ${pi}"/>
+            <origin xyz="0 0 0" rpy="0 0 0"/>
         </xacro:inertial_cylinder>
     </link>
@@ -83,5 +83,5 @@
         </collision>
         <xacro:inertial_cylinder mass="0.05" length="${wheel_thickness}" radius="${wheel_radius}">
-            <origin xyz="0 0.10575 -0.0225" rpy="${-pi/2} ${pi/2} 0"/>
+            <origin xyz="0 0 0" rpy="0 0 0"/>
         </xacro:inertial_cylinder>
     </link>
@@ -92,9 +92,9 @@
         <child link="U_base_wheel_1_link"/>
         <axis xyz="0 0 -1"/>
-        <limit effort="0.323" velocity="10.47" />
+        <limit effort="0" velocity="0" />
     </joint>
     <xacro:property name="U_base_box_X" value="0.028"/>
     <xacro:property name="U_base_box_Y" value="0.032"/>
-    <xacro:property name="U_base_box_Z" value="0.04402"/>
+    <xacro:property name="U_base_box_Z" value="0.044"/>
     <link name="U_base_wheel_1_link">
         <visual>
@@ -112,5 +112,5 @@
         </collision>
         <xacro:inertial_box mass="0.0125" x="${U_base_box_X}" y="${U_base_box_Y}" z="${U_base_box_Z}">
-            <origin xyz="0.05751 0 -0.0278" rpy="${pi} 0 0"/>
+            <origin xyz="0 0 0" rpy="0 0 0"/>
         </xacro:inertial_box>
     </link>
@@ -121,5 +121,5 @@
         <child link="U_wheel_1_link"/>
         <axis xyz="0 0 1"/>
-        <limit effort="0.323" velocity="10.47" />
+        <limit effort="0" velocity="0" />
     </joint>
     <xacro:property name="U_wheel_thickness" value="0.0144"/>
@@ -140,5 +140,5 @@
         </collision>
         <xacro:inertial_cylinder mass="0.005" length="${U_wheel_thickness}" radius="${U_wheel_radius}">
-            <origin xyz="0.01577 0 0.01622" rpy="${pi/2} 0 ${pi/2}"/>
+            <origin xyz="0 0 0" rpy="0 0 0"/>
         </xacro:inertial_cylinder>
     </link>
@@ -149,5 +149,5 @@
         <child link="U_base_wheel_2_link"/>
         <axis xyz="0 0 -1"/>
-        <limit effort="0.323" velocity="10.47" />
+        <limit effort="0" velocity="0" />
     </joint>
     <link name="U_base_wheel_2_link">
@@ -166,5 +166,5 @@
         </collision>
         <xacro:inertial_box mass="0.0125" x="${U_base_box_X}" y="${U_base_box_Y}" z="${U_base_box_Z}">
-            <origin xyz="-0.05751 0 -0.0278" rpy="${pi} 0 0"/>
+            <origin xyz="0 0 0" rpy="0 0 0"/>
         </xacro:inertial_box>
     </link>
@@ -175,5 +175,5 @@
         <child link="U_wheel_2_link"/>
         <axis xyz="0 0 1"/>
-        <limit effort="0.323" velocity="10.47" />
+        <limit effort="0" velocity="0" />
     </joint>
     <link name="U_wheel_2_link">
@@ -192,5 +192,31 @@
         </collision>
         <xacro:inertial_cylinder mass="0.005" length="${U_wheel_thickness}" radius="${U_wheel_radius}">
-            <origin xyz="0.01577 0 0.01622" rpy="${pi/2} 0 ${pi/2}"/>
+            <origin xyz="0 0 0" rpy="0 0 0"/>
+        </xacro:inertial_cylinder>
+    </link>
+    <!--Fixed support-->
+    <joint name="Support_joint" type="fixed">
+        <origin xyz="0 0 0.101" rpy="0 0 0"/>
+        <parent link="B_base_link"/>
+        <child link="Support_link"/>
+    </joint>
+    <xacro:property name="Support_length" value="0.101"/>
+    <xacro:property name="Support_radius" value="0.070"/>
+    <link name="Support_link">
+        <visual>
+            <origin xyz="0 0 -${Support_length/2}" rpy="0 0 0"/>
+            <geometry>
+                <cylinder length="${Support_length}" radius="${Support_radius}"/>
+            </geometry>
+            <material name="white"/>
+        </visual>
+        <collision>
+            <origin xyz="0 0 -${Support_length/2}" rpy="0 0 0"/>
+            <geometry>
+                <cylinder length="${Support_length}" radius="${Support_radius}"/>
+            </geometry>
+        </collision>
+        <xacro:inertial_cylinder mass="0.5" length="${Support_length}" radius="${Support_radius}">
+            <origin xyz="0 0 -${Support_length/2}" rpy="0 0 0"/>
         </xacro:inertial_cylinder>
     </link>

File: install/robot_pkg/share/robot_pkg/urdf/gazebo_setup.xacro (robot description, xacro)
@@ -24,9 +24,8 @@
     </gazebo>
     <gazebo reference="Support_link">
-      <material>Gazebo/Yellow</material>
+      <material>Gazebo/White</material>
     </gazebo>
     <!-- Define friction for wheels -->
     <gazebo reference="L_wheel_link">
-        <material>Gazebo/Black</material>
         <surface>
             <friction>
@@ -39,5 +38,4 @@
     </gazebo>
     <gazebo reference="R_wheel_link">
-        <material>Gazebo/Black</material>
         <surface>
             <friction>
@@ -49,4 +47,45 @@
         </surface>
     </gazebo>
+    <!-- Define friction for caster wheels -->
+    <gazebo reference="U_base_wheel_1_joint">
+      <surface>
+          <friction>
+              <ode>
+                  <mu>0.001</mu>
+                  <mu2>0.001</mu2>
+              </ode>
+          </friction>
+      </surface>
+  </gazebo>
+  <gazebo reference="U_wheel_1_joint">
+    <surface>
+        <friction>
+            <ode>
+                <mu>0.2</mu>
+                <mu2>0.2</mu2>
+            </ode>
+        </friction>
+    </surface>
+</gazebo>
+<gazebo reference="U_base_wheel_2_joint">
+  <surface>
+      <friction>
+          <ode>
+              <mu>0.001</mu>
+              <mu2>0.001</mu2>
+          </ode>
+      </friction>
+  </surface>
+</gazebo>
+<gazebo reference="U_wheel_2_joint">
+<surface>
+    <friction>
+        <ode>
+            <mu>0.2</mu>
+            <mu2>0.2</mu2>
+        </ode>
+    </friction>
+</surface>
+</gazebo>
     <!-- Define plugins -->
     <gazebo>

Commit message: final urdf

File: install/robot_pkg/share/robot_pkg/urdf/TTR01.urdf.xacro (robot description, xacro)
@@ -1 +1 @@
-/home/dev-pc/dev_ws/src/robot_pkg/urdf/TTR01.urdf.xacro
+/home/rodrigo/dev_ws/src/robot_pkg/urdf/TTR01.urdf.xacro

File: install/robot_pkg/share/robot_pkg/urdf/gazebo_setup.xacro (robot description, xacro)
@@ -1 +1 @@
-/home/dev-pc/dev_ws/src/robot_pkg/urdf/gazebo_setup.xacro
+/home/rodrigo/dev_ws/src/robot_pkg/urdf/gazebo_setup.xacro

File: install/robot_pkg/share/robot_pkg/urdf/robot_parameters.xacro (robot description, xacro)
@@ -1 +1 @@
-/home/dev-pc/dev_ws/src/robot_pkg/urdf/robot_parameters.xacro
+/home/rodrigo/dev_ws/src/robot_pkg/urdf/robot_parameters.xacro

File: src/robot_pkg/urdf/TTR01.urdf.xacro (robot description, xacro)
@@ -1,6 +1,6 @@
 <?xml version="1.0"?>
 <robot xmlns:xacro="http://www.ros.org/wiki/xacro"  name="TTR01">
+    <xacro:include filename="robot_parameters.xacro"/>
     <!--base/world frame-->
-    <xacro:include filename="robot_parameters.xacro"/>
     <link name="base_link"> </link>
     <!--Bottom base frame-->
@@ -34,5 +34,5 @@
     <!--Left wheel frame-->
     <joint name="L_wheel_joint" type="continuous">
-        <origin xyz="0 -0.10575 -0.0225" rpy="${-pi/2} ${-pi/2} ${pi}"/>
+        <origin xyz="0 -0.10575 -0.02356" rpy="${pi/2} ${pi/2} 0"/>
         <parent link="B_base_link"/>
         <child link="L_wheel_link"/>
@@ -62,5 +62,5 @@
     <!--Right wheel frame-->
     <joint name="R_wheel_joint" type="continuous">
-        <origin xyz="0 0.10575 -0.0225" rpy="${-pi/2} ${pi/2} 0"/>
+        <origin xyz="0 0.10575 -0.02356" rpy="${-pi/2} ${pi/2} 0"/>
         <parent link="B_base_link"/>
         <child link="R_wheel_link"/>
@@ -91,13 +91,12 @@
         <parent link="B_base_link"/>
         <child link="U_base_wheel_1_link"/>
-        <axis xyz="0 0 -1"/>
-        <limit effort="0" velocity="0" />
+        <axis xyz="0 0 1"/>
     </joint>
     <xacro:property name="U_base_box_X" value="0.028"/>
     <xacro:property name="U_base_box_Y" value="0.032"/>
-    <xacro:property name="U_base_box_Z" value="0.045"/>
+    <xacro:property name="U_base_box_Z" value="0.03902"/>
     <link name="U_base_wheel_1_link">
         <visual>
-            <origin xyz="0 0 0" rpy="0 0 0"/>
+            <origin xyz="0 0 -0.00329" rpy="0 0 0"/>
             <geometry>
                 <box size="${U_base_box_X} ${U_base_box_Y} ${U_base_box_Z}"/>
@@ -106,5 +105,5 @@
         </visual>
         <collision>
-            <origin xyz="0 0 0" rpy="0 0 0"/>
+            <origin xyz="0 0 -0.00329" rpy="0 0 0"/>
             <geometry>
                 <box size="${U_base_box_X} ${U_base_box_Y} ${U_base_box_Z}"/>
@@ -121,5 +120,4 @@
         <child link="U_wheel_1_link"/>
         <axis xyz="0 0 1"/>
-        <limit effort="0" velocity="0" />
     </joint>
     <xacro:property name="U_wheel_thickness" value="0.0144"/>
@@ -148,10 +146,10 @@
         <parent link="B_base_link"/>
         <child link="U_base_wheel_2_link"/>
-        <axis xyz="0 0 -1"/>
+        <axis xyz="0 0 1"/>
         <limit effort="0" velocity="0" />
     </joint>
     <link name="U_base_wheel_2_link">
         <visual>
-            <origin xyz="0 0 0" rpy="0 0 0"/>
+            <origin xyz="0 0 -0.00329" rpy="0 0 0"/>
             <geometry>
                 <box size="${U_base_box_X} ${U_base_box_Y} ${U_base_box_Z}"/>
@@ -160,5 +158,5 @@
         </visual>
         <collision>
-            <origin xyz="0 0 0" rpy="0 0 0"/>
+            <origin xyz="0 0 -0.00329" rpy="0 0 0"/>
             <geometry>
                 <box size="${U_base_box_X} ${U_base_box_Y} ${U_base_box_Z}"/>

File: src/robot_pkg/urdf/gazebo_setup.xacro (robot description, xacro)
@@ -62,6 +62,6 @@
         <friction>
             <ode>
-                <mu>0.2</mu>
-                <mu2>0.2</mu2>
+                <mu>0.3</mu>
+                <mu2>0.3</mu2>
             </ode>
         </friction>
@@ -82,6 +82,6 @@
     <friction>
         <ode>
-            <mu>0.2</mu>
-            <mu2>0.2</mu2>
+            <mu>0.3</mu>
+            <mu2>0.3</mu2>
         </ode>
     </friction>
