Commit message: gazebo sim

File: install/robot_pkg/share/robot_pkg/urdf/gazebo_control.xacro (robot description, xacro)
@@ -1 +1 @@
-/home/rodrigo/dev_ws/src/robot_pkg/urdf/gazebo_control.xacro
+/home/dev-pc/dev_ws/src/robot_pkg/urdf/gazebo_control.xacro

File: install/robot_pkg/share/robot_pkg/urdf/ros2_control.xacro (robot description, xacro)
@@ -1 +1 @@
-/home/rodrigo/dev_ws/src/robot_pkg/urdf/ros2_control.xacro
+/home/dev-pc/dev_ws/src/robot_pkg/urdf/ros2_control.xacro

File: src/robot_pkg/urdf/gazebo_setup.xacro (robot description, xacro)
@@ -66,5 +66,5 @@
     </gazebo>
     <!-- Define friction for caster wheels -->
-    <!-- <gazebo reference="U_base_wheel_1_joint">
+    <gazebo reference="U_base_wheel_1_joint">
       <surface>
           <friction>
@@ -75,5 +75,5 @@
           </friction>
       </surface>
-  </gazebo> -->
+  </gazebo>
   <gazebo reference="U_wheel_1_joint">
     <surface>
@@ -86,5 +86,5 @@
     </surface>
 </gazebo>
-<!-- <gazebo reference="U_base_wheel_2_joint">
+<gazebo reference="U_base_wheel_2_joint">
   <surface>
       <friction>
@@ -95,5 +95,5 @@
       </friction>
   </surface>
-</gazebo> -->
+</gazebo>
 <gazebo reference="U_wheel_2_joint">
 <surface>
@@ -112,8 +112,8 @@
             <joint_name>L_wheel_joint</joint_name>
             <joint_name>R_wheel_joint</joint_name>
-            <!-- <joint_name>U_base_wheel_1_joint</joint_name>
+            <joint_name>U_base_wheel_1_joint</joint_name>
             <joint_name>U_wheel_1_joint</joint_name>
             <joint_name>U_base_wheel_2_joint</joint_name>
-            <joint_name>U_wheel_2_joint</joint_name> -->
+            <joint_name>U_wheel_2_joint</joint_name>
              <joint_name>Lidar_motor_joint</joint_name>
         </plugin>

File: src/robot_pkg/urdf/robot.xacro (robot description, xacro)
@@ -82,9 +82,9 @@
     </link>
     <!--Caster wheel base 1-->
-    <joint name="U_base_wheel_1_joint" type="fixed">
+    <joint name="U_base_wheel_1_joint" type="continuous">
         <origin xyz="0.05751 0 -0.0278" rpy="${pi} 0 0"/>
         <parent link="B_base_link"/>
         <child link="U_base_wheel_1_link"/>
-        <!-- <axis xyz="0 0 1"/> -->
+        <axis xyz="0 0 1"/>
     </joint>
     <link name="U_base_wheel_1_link">
@@ -107,9 +107,9 @@
     </link>
     <!--Caster wheel 1-->
-    <joint name="U_wheel_1_joint" type="fixed">
+    <joint name="U_wheel_1_joint" type="continuous">
         <origin xyz="0.01577 0 0.01622" rpy="${pi/2} 0 0"/>
         <parent link="U_base_wheel_1_link"/>
         <child link="U_wheel_1_link"/>
-        <!-- <axis xyz="0 0 -1"/>    -->
+        <axis xyz="0 0 -1"/>
     </joint>
     <link name="U_wheel_1_link">
@@ -132,9 +132,9 @@
     </link>
     <!--Caster wheel base 2-->
-    <joint name="U_base_wheel_2_joint" type="fixed">
+    <joint name="U_base_wheel_2_joint" type="continuous">
         <origin xyz="-0.05751 0 -0.0278" rpy="${pi} 0 ${pi}"/>
         <parent link="B_base_link"/>
         <child link="U_base_wheel_2_link"/>
-        <!-- <axis xyz="0 0 -1"/> -->
+        <axis xyz="0 0 -1"/>
     </joint>
     <link name="U_base_wheel_2_link">
@@ -157,9 +157,9 @@
     </link>
     <!--Caster wheel 2-->
-    <joint name="U_wheel_2_joint" type="fixed">
+    <joint name="U_wheel_2_joint" type="continuous">
         <origin xyz="0.01577 0 0.01622" rpy="${pi/2} 0 0"/>
         <parent link="U_base_wheel_2_link"/>
         <child link="U_wheel_2_link"/>
-        <!-- <axis xyz="0 0 1"/>   -->
+        <axis xyz="0 0 1"/>
     </joint>
     <link name="U_wheel_2_link">

File: src/robot_pkg/urdf/ros2_control.xacro (robot description, xacro)
@@ -1,5 +1,5 @@
 <?xml version="1.0"?>
 <robot xmlns:xacro="http://www.ros.org/wiki/xacro">
-    <ros2_control name="RealRobot" type="system">
+    <!-- <ros2_control name="RealRobot" type="system">
         <hardware>
             <plugin>diffdrive_arduino/DiffDriveArduino</plugin>
@@ -28,6 +28,6 @@
             <state_interface name="position"/>
         </joint>
-    </ros2_control>
-    <!-- <ros2_control name="GazeboSystem" type="system">
+    </ros2_control> -->
+    <ros2_control name="GazeboSystem" type="system">
         <hardware>
             <plugin>gazebo_ros2_control/GazeboSystem</plugin>
@@ -54,5 +54,5 @@
                 <parameters> $(find robot_pkg)/config/controllers.yaml </parameters>
             </plugin>
-    </gazebo> -->
+    </gazebo>
+</robot>
     <!-- ros2 run controller_manager_ros_control_node -->
-</robot>

Commit message: good control bad rviz

File: install/robot_pkg/share/robot_pkg/urdf/gazebo_control.xacro (robot description, xacro)
@@ -1 +1 @@
-/home/dev-pc/dev_ws/src/robot_pkg/urdf/gazebo_control.xacro
+/home/rodrigo/dev_ws/src/robot_pkg/urdf/gazebo_control.xacro

File: install/robot_pkg/share/robot_pkg/urdf/ros2_control.xacro (robot description, xacro)
@@ -1 +1 @@
-/home/dev-pc/dev_ws/src/robot_pkg/urdf/ros2_control.xacro
+/home/rodrigo/dev_ws/src/robot_pkg/urdf/ros2_control.xacro

File: src/robot_pkg/urdf/robot.xacro (robot description, xacro)
@@ -34,5 +34,5 @@
         <parent link="B_base_link"/>
         <child link="L_wheel_link"/>
-        <axis xyz="0 0 -1"/>
+        <axis xyz="0 0 1"/>
         <limit effort="0.323" velocity="10.47" />
     </joint>
@@ -60,5 +60,5 @@
         <parent link="B_base_link"/>
         <child link="R_wheel_link"/>
-        <axis xyz="0 0 1"/>
+        <axis xyz="0 0 -1"/>
         <limit effort="0.323" velocity="10.47" />
     </joint>

File: src/robot_pkg/urdf/ros2_control.xacro (robot description, xacro)
@@ -1,14 +1,14 @@
 <?xml version="1.0"?>
 <robot xmlns:xacro="http://www.ros.org/wiki/xacro">
-    <!-- <ros2_control name="RealRobot" type="system">
+    <ros2_control name="RealRobot" type="system">
         <hardware>
             <plugin>diffdrive_arduino/DiffDriveArduino</plugin>
-            <param name="left_wheel_name">L_wheel_joint</param>
-            <param name="right_wheel_name">R_wheel_joint</param>
+            <param name="left_wheel_name">R_wheel_joint</param>
+            <param name="right_wheel_name">L_wheel_joint</param>
             <param name="loop_rate">30</param>
             <param name="device">/dev/ttyUSB1</param>
             <param name="baud_rate">57600</param>
-            <param name="timeout">1400</param>
-            <param name="enc_counts_per_rev">2491</param>
+            <param name="timeout">1000</param>
+            <param name="enc_counts_per_rev">1758</param>
         </hardware>
         <joint name="L_wheel_joint">
@@ -28,6 +28,6 @@
             <state_interface name="position"/>
         </joint>
-    </ros2_control> -->
-    <ros2_control name="GazeboSystem" type="system">
+    </ros2_control>
+    <!-- <ros2_control name="GazeboSystem" type="system">
         <hardware>
             <plugin>gazebo_ros2_control/GazeboSystem</plugin>
@@ -54,5 +54,5 @@
                 <parameters> $(find robot_pkg)/config/controllers.yaml </parameters>
             </plugin>
-    </gazebo>
+    </gazebo> -->
 </robot>
     <!-- ros2 run controller_manager_ros_control_node -->
