Commit message: diff drive complete

File: src/robot_pkg/urdf/gazebo_control.xacro (robot description, xacro)
@@ -8,5 +8,5 @@
             <left_joint>L_wheel_joint</left_joint>
             <right_joint>R_wheel_joint</right_joint>
-            <wheel_separation>0.2115</wheel_separation> <!-- Adjust according to your robot -->
+            <wheel_separation>0.208</wheel_separation> <!-- Adjust according to your robot -->
             <wheel_diameter>0.065</wheel_diameter> <!-- Adjust according to your wheels -->
             <!-- Limits -->

File: src/robot_pkg/urdf/robot.xacro (robot description, xacro)
@@ -31,5 +31,5 @@
     <!--Left wheel-->
     <joint name="L_wheel_joint" type="continuous">
-        <origin xyz="0 -0.10575 -0.02356" rpy="${pi/2} ${pi/2} 0"/>
+        <origin xyz="0 -0.104 -0.02356" rpy="${pi/2} ${pi/2} 0"/>
         <parent link="B_base_link"/>
         <child link="L_wheel_link"/>
@@ -57,5 +57,5 @@
     <!--Right wheel-->
     <joint name="R_wheel_joint" type="continuous">
-        <origin xyz="0 0.10575 -0.02356" rpy="${-pi/2} ${pi/2} 0"/>
+        <origin xyz="0 0.104 -0.02356" rpy="${-pi/2} ${pi/2} 0"/>
         <parent link="B_base_link"/>
         <child link="R_wheel_link"/>

File: src/robot_pkg/urdf/ros2_control.xacro (robot description, xacro)
@@ -4,11 +4,11 @@
         <hardware>
             <plugin>diffdrive_arduino/DiffDriveArduino</plugin>
-            <param name="left_wheel_name">R_wheel_joint</param>
-            <param name="right_wheel_name">L_wheel_joint</param>
+            <param name="left_wheel_name">L_wheel_joint</param>
+            <param name="right_wheel_name">R_wheel_joint</param>
             <param name="loop_rate">30</param>
             <param name="device">/dev/ttyUSB1</param>
             <param name="baud_rate">57600</param>
             <param name="timeout">1000</param>
-            <param name="enc_counts_per_rev">1758</param>
+            <param name="enc_counts_per_rev">2500</param>
         </hardware>
         <joint name="L_wheel_joint">

Commit message: almost gazebo

File: src/robot_pkg/urdf/gazebo_control.xacro (robot description, xacro)
@@ -9,5 +9,5 @@
             <right_joint>R_wheel_joint</right_joint>
             <wheel_separation>0.208</wheel_separation> <!-- Adjust according to your robot -->
-            <wheel_diameter>0.065</wheel_diameter> <!-- Adjust according to your wheels -->
+            <wheel_diameter>0.0682</wheel_diameter> <!-- Adjust according to your wheels -->
             <!-- Limits -->
             <max_wheel_torque>0.5</max_wheel_torque>

File: src/robot_pkg/urdf/gazebo_setup.xacro (robot description, xacro)
@@ -38,4 +38,7 @@
       <material>Gazebo/White</material>
     </gazebo>
+    <gazebo reference="Lidar_motor_link">
+      <material>Gazebo/Black</material>
+    </gazebo>
     <gazebo reference="Camera_base_link">
       <material>Gazebo/Black</material>
@@ -49,6 +52,6 @@
             <friction>
                 <ode>
-                    <mu>1.0</mu>
-                    <mu2>1.0</mu2>
+                    <mu>0.6</mu>
+                    <mu2>0.6</mu2>
                 </ode>
             </friction>
@@ -59,6 +62,6 @@
             <friction>
                 <ode>
-                    <mu>1.0</mu>
-                    <mu2>1.0</mu2>
+                    <mu>0.6</mu>
+                    <mu2>0.6</mu2>
                 </ode>
             </friction>
@@ -70,6 +73,6 @@
           <friction>
               <ode>
-                  <mu>0.1</mu>
-                  <mu2>0.1</mu2>
+                  <mu>0.001</mu>
+                  <mu2>0.001</mu2>
               </ode>
           </friction>
@@ -80,6 +83,6 @@
         <friction>
             <ode>
-                <mu>0.3</mu>
-                <mu2>0.3</mu2>
+                <mu>0.01</mu>
+                <mu2>0.01</mu2>
             </ode>
         </friction>
@@ -90,6 +93,6 @@
       <friction>
           <ode>
-              <mu>0.1</mu>
-              <mu2>0.1</mu2>
+              <mu>0.001</mu>
+              <mu2>0.001</mu2>
           </ode>
       </friction>
@@ -100,6 +103,6 @@
     <friction>
         <ode>
-            <mu>0.3</mu>
-            <mu2>0.3</mu2>
+            <mu>0.01</mu>
+            <mu2>0.01</mu2>
         </ode>
     </friction>

File: src/robot_pkg/urdf/lidar.xacro (robot description, xacro)
@@ -30,5 +30,5 @@
         <parent link="Lidar_base_link"/>
         <child link="Lidar_motor_link"/>
-        <axis xyz="0 0 1"/>
+        <axis xyz="0 0 -1"/>
     </joint>
     <link name="Lidar_motor_link">

File: src/robot_pkg/urdf/robot.xacro (robot description, xacro)
@@ -1,5 +1,5 @@
 <?xml version="1.0"?>
 <robot xmlns:xacro="http://www.ros.org/wiki/xacro" >
-    <!--base/world-->
+    <!--base link-->
     <link name="base_link"> </link>
     <!--Bottom base-->
@@ -31,6 +31,6 @@
     <!--Left wheel-->
     <joint name="L_wheel_joint" type="continuous">
-        <origin xyz="0 -0.104 -0.02356" rpy="${pi/2} ${pi/2} 0"/>
-        <parent link="B_base_link"/>
+        <origin xyz="0 0.104 0" rpy="-${pi/2} ${pi/2} 0"/>
+        <parent link="base_link"/>
         <child link="L_wheel_link"/>
         <axis xyz="0 0 1"/>
@@ -57,38 +57,62 @@
     <!--Right wheel-->
     <joint name="R_wheel_joint" type="continuous">
-        <origin xyz="0 0.104 -0.02356" rpy="${-pi/2} ${pi/2} 0"/>
+        <origin xyz="0 -0.104 0" rpy="${pi/2} ${pi/2} 0"/>
+        <parent link="base_link"/>
+        <child link="R_wheel_link"/>
+        <axis xyz="0 0 -1"/>
+        <limit effort="0.323" velocity="10.47" />
+    </joint>
+    <link name="R_wheel_link">
+        <visual>
+            <origin xyz="0 0 0" rpy="0 0 0"/>
+            <geometry>
+                <cylinder length="${wheel_thickness}" radius="${wheel_radius}"/>
+            </geometry>
+            <material name="black"/>
+        </visual>
+        <collision>
+            <origin xyz="0 0 0" rpy="0 0 0"/>
+            <geometry>
+                <cylinder length="${wheel_thickness}" radius="${wheel_radius}"/>
+            </geometry>
+        </collision>
+        <xacro:inertial_cylinder mass="${wheel_mass}" length="${wheel_thickness}" radius="${wheel_radius}">
+            <origin xyz="0 0 0" rpy="0 0 0"/>
+        </xacro:inertial_cylinder>
+    </link>
+    <!-- Caster support 1 -->
+    <joint name="C_support_1_joint" type="fixed">
+        <origin xyz="0.05751 0 -0.005" rpy="0 0 0"/>
         <parent link="B_base_link"/>
-        <child link="R_wheel_link"/>
-        <axis xyz="0 0 -1"/>
-        <limit effort="0.323" velocity="10.47" />
-    </joint>
-    <link name="R_wheel_link">
-        <visual>
-            <origin xyz="0 0 0" rpy="0 0 0"/>
-            <geometry>
-                <cylinder length="${wheel_thickness}" radius="${wheel_radius}"/>
-            </geometry>
-            <material name="black"/>
-        </visual>
-        <collision>
-            <origin xyz="0 0 0" rpy="0 0 0"/>
-            <geometry>
-                <cylinder length="${wheel_thickness}" radius="${wheel_radius}"/>
-            </geometry>
-        </collision>
-        <xacro:inertial_cylinder mass="${wheel_mass}" length="${wheel_thickness}" radius="${wheel_radius}">
-            <origin xyz="0 0 0" rpy="0 0 0"/>
-        </xacro:inertial_cylinder>
+        <child link="C_support_1_link"/>
+    </joint>
+    <link name="C_support_1_link">
+        <visual>
+            <origin xyz="0 0 -${C_support_box_Z/2}" rpy="0 0 0"/>
+            <geometry>
+                <box size="${C_support_box_X} ${C_support_box_Y} ${C_support_box_Z}"/>
+            </geometry>
+            <material name="white"/>
+        </visual>
+        <collision>
+            <origin xyz="0 0 -${C_support_box_Z/2}" rpy="0 0 0"/>
+            <geometry>
+                <box size="${C_support_box_X} ${C_support_box_Y} ${C_support_box_Z}"/>
+            </geometry>
+        </collision>
+        <xacro:inertial_box mass="${C_support_mass}" x="${C_support_box_X}" y="${C_support_box_Y}" z="${C_support_box_Z}">
+            <origin xyz="0 0 -${C_support_box_Z/2}" rpy="0 0 0"/>
+        </xacro:inertial_box>
     </link>
     <!--Caster wheel base 1-->
     <joint name="U_base_wheel_1_joint" type="continuous">
-        <origin xyz="0.05751 0 -0.0278" rpy="${pi} 0 0"/>
-        <parent link="B_base_link"/>
+        <origin xyz="0 0 -0.013" rpy="${pi} 0 0"/>
+        <parent link="C_support_1_link"/>
         <child link="U_base_wheel_1_link"/>
-        <axis xyz="0 0 1"/>
+        <axis xyz="0 0 -1"/>
     </joint>
     <link name="U_base_wheel_1_link">
         <visual>
-            <origin xyz="0 0 -0.00329" rpy="0 0 0"/>
+            <origin xyz="0 0 ${U_base_box_Z/2}" rpy="0 0 0"/>
             <geometry>
                 <box size="${U_base_box_X} ${U_base_box_Y} ${U_base_box_Z}"/>
@@ -97,5 +121,5 @@
         </visual>
         <collision>
-            <origin xyz="0 0 -0.00329" rpy="0 0 0"/>
+            <origin xyz="0 0 ${U_base_box_Z/2}" rpy="0 0 0"/>
             <geometry>
                 <box size="${U_base_box_X} ${U_base_box_Y} ${U_base_box_Z}"/>
@@ -103,10 +127,10 @@
         </collision>
         <xacro:inertial_box mass="${U_base_mass}" x="${U_base_box_X}" y="${U_base_box_Y}" z="${U_base_box_Z}">
-            <origin xyz="0 0 -0.00329" rpy="0 0 0"/>
+            <origin xyz="0 0 ${U_base_box_Z/2}" rpy="0 0 0"/>
         </xacro:inertial_box>
     </link>
     <!--Caster wheel 1-->
     <joint name="U_wheel_1_joint" type="continuous">
-        <origin xyz="0.01577 0 0.01622" rpy="${pi/2} 0 0"/>
+        <origin xyz="0.016 0 0.0256" rpy="${pi/2} 0 0"/>
         <parent link="U_base_wheel_1_link"/>
         <child link="U_wheel_1_link"/>
@@ -131,8 +155,32 @@
         </xacro:inertial_cylinder>
     </link>
+    <!-- Caster support 2 -->
+    <joint name="C_support_2_joint" type="fixed">
+        <origin xyz="-0.05751 0 -0.005" rpy="0 0 0"/>
+        <parent link="B_base_link"/>
+        <child link="C_support_2_link"/>
+    </joint>
+    <link name="C_support_2_link">
+        <visual>
+            <origin xyz="0 0 -${C_support_box_Z/2}" rpy="0 0 0"/>
+            <geometry>
+                <box size="${C_support_box_X} ${C_support_box_Y} ${C_support_box_Z}"/>
+            </geometry>
+            <material name="white"/>
+        </visual>
+        <collision>
+            <origin xyz="0 0 -${C_support_box_Z/2}" rpy="0 0 0"/>
+            <geometry>
+                <box size="${C_support_box_X} ${C_support_box_Y} ${C_support_box_Z}"/>
+            </geometry>
+        </collision>
+        <xacro:inertial_box mass="${C_support_mass}" x="${C_support_box_X}" y="${C_support_box_Y}" z="${C_support_box_Z}">
+            <origin xyz="0 0 -${C_support_box_Z/2}" rpy="0 0 0"/>
+        </xacro:inertial_box>
+    </link>
     <!--Caster wheel base 2-->
     <joint name="U_base_wheel_2_joint" type="continuous">
-        <origin xyz="-0.05751 0 -0.0278" rpy="${pi} 0 ${pi}"/>
-        <parent link="B_base_link"/>
+        <origin xyz="0 0 -0.013" rpy="${pi} 0 0"/>
+        <parent link="C_support_2_link"/>
         <child link="U_base_wheel_2_link"/>
         <axis xyz="0 0 -1"/>
@@ -140,5 +188,5 @@
     <link name="U_base_wheel_2_link">
         <visual>
-            <origin xyz="0 0 -0.00329" rpy="0 0 0"/>
+            <origin xyz="0 0 ${U_base_box_Z/2}" rpy="0 0 0"/>
             <geometry>
                 <box size="${U_base_box_X} ${U_base_box_Y} ${U_base_box_Z}"/>
@@ -147,5 +195,5 @@
         </visual>
         <collision>
-            <origin xyz="0 0 -0.00329" rpy="0 0 0"/>
+            <origin xyz="0 0 ${U_base_box_Z/2}" rpy="0 0 0"/>
             <geometry>
                 <box size="${U_base_box_X} ${U_base_box_Y} ${U_base_box_Z}"/>
@@ -153,13 +201,13 @@
         </collision>
         <xacro:inertial_box mass="${U_base_mass}" x="${U_base_box_X}" y="${U_base_box_Y}" z="${U_base_box_Z}">
-            <origin xyz="0 0 -0.00329" rpy="0 0 0"/>
+            <origin xyz="0 0 ${U_base_box_Z/2}" rpy="0 0 0"/>
         </xacro:inertial_box>
     </link>
     <!--Caster wheel 2-->
     <joint name="U_wheel_2_joint" type="continuous">
-        <origin xyz="0.01577 0 0.01622" rpy="${pi/2} 0 0"/>
+        <origin xyz="0.016 0 0.0256" rpy="${pi/2} 0 0"/>
         <parent link="U_base_wheel_2_link"/>
         <child link="U_wheel_2_link"/>
-        <axis xyz="0 0 1"/>
+        <axis xyz="0 0 -1"/>
     </joint>
     <link name="U_wheel_2_link">
@@ -249,5 +297,5 @@
             </geometry>
         </collision>
-        <xacro:inertial_box mass="${Support_B_mass}" x="${Support_BX}" y="${Support_BY}" z="${Support_AZ}">
+        <xacro:inertial_box mass="${Support_B_mass}" x="${Support_BX}" y="${Support_BY}" z="${Support_BZ}">
             <origin xyz="0 0 0" rpy="0 0 0"/>
         </xacro:inertial_box>

File: src/robot_pkg/urdf/robot_parameters.xacro (robot description, xacro)
@@ -35,10 +35,13 @@
     <xacro:property name="Support_BZ" value="0.051"/>
     <xacro:property name="wheel_thickness" value="0.027"/>
-    <xacro:property name="wheel_radius" value="0.0325"/>
+    <xacro:property name="wheel_radius" value="0.0341"/>
+    <xacro:property name="C_support_box_X" value="0.032"/>
+    <xacro:property name="C_support_box_Y" value="0.038"/>
+    <xacro:property name="C_support_box_Z" value="0.013"/>
     <xacro:property name="U_base_box_X" value="0.032"/>
     <xacro:property name="U_base_box_Y" value="0.038"/>
-    <xacro:property name="U_base_box_Z" value="0.03902"/>
+    <xacro:property name="U_base_box_Z" value="0.0256"/>
     <xacro:property name="U_wheel_thickness" value="0.0144"/>
-    <xacro:property name="U_wheel_radius" value="0.0115"/>
+    <xacro:property name="U_wheel_radius" value="0.013"/>
     <xacro:property name="Lidar_base_X" value="0.10457"/>
     <xacro:property name="Lidar_base_Y" value="0.0787"/>
@@ -56,6 +59,7 @@
     <xacro:property name="MT_mass" value="0.04"/>
     <xacro:property name="Support_A_mass" value="0.3"/>
-    <xacro:property name="Support_B_mass" value="0.5"/>
-    <xacro:property name="wheel_mass" value="0.120"/>
+    <xacro:property name="Support_B_mass" value="0.3"/>
+    <xacro:property name="wheel_mass" value="0.300"/>
+    <xacro:property name="C_support_mass" value="0.01"/>
     <xacro:property name="U_base_mass" value="0.05"/>
     <xacro:property name="U_wheel_mass" value="0.01"/>
@@ -88,6 +92,6 @@
             <mass value="${mass}" />
             <inertia ixx="${(1/12) * mass * (3*radius*radius + length*length)}" ixy="0.0" ixz="0.0"
-                    iyy="${(1/12) * mass * (3*radius*radius + length*length)}" iyz="0.0"
-                    izz="${(1/2) * mass * (radius*radius)}" />
+                    iyy="${(1/2) * mass * (radius*radius)}"
+                    izz="${(1/12) * mass * (3*radius*radius + length*length)}" iyz="0.0" />
         </inertial>
     </xacro:macro>

File: src/robot_pkg/urdf/ros2_control.xacro (robot description, xacro)
@@ -1,5 +1,5 @@
 <?xml version="1.0"?>
 <robot xmlns:xacro="http://www.ros.org/wiki/xacro">
-    <ros2_control name="RealRobot" type="system">
+    <!-- <ros2_control name="RealRobot" type="system">
         <hardware>
             <plugin>diffdrive_arduino/DiffDriveArduino</plugin>
@@ -20,5 +20,5 @@
             <state_interface name="position"/>
         </joint>
-        <joint name="L_wheel_joint">
+        <joint name="R_wheel_joint">
             <command_interface name="velocity">
                 <param name="min">-10</param>
@@ -28,10 +28,10 @@
             <state_interface name="position"/>
         </joint>
-    </ros2_control>
-    <!-- <ros2_control name="GazeboSystem" type="system">
+    </ros2_control> -->
+    <ros2_control name="GazeboSystem" type="system">
         <hardware>
             <plugin>gazebo_ros2_control/GazeboSystem</plugin>
         </hardware>
-        <joint name="L_wheel_joint">
+        <joint name="R_wheel_joint">
             <command_interface name="velocity">
                 <param name="min">-10</param>
@@ -41,5 +41,5 @@
             <state_interface name="velocity" />
         </joint>
-        <joint name="R_wheel_joint">
+        <joint name="L_wheel_joint">
             <command_interface name="velocity">
                 <param name="min">-10</param>
@@ -54,5 +54,5 @@
                 <parameters> $(find robot_pkg)/config/controllers.yaml </parameters>
             </plugin>
-    </gazebo> -->
+    </gazebo>
 </robot>
     <!-- ros2 run controller_manager_ros_control_node -->
