Commit message: main urdf

File: src/robot_pkg/urdf/TTR01.urdf.xacro (robot description, xacro)
@@ -2,221 +2,5 @@
 <robot xmlns:xacro="http://www.ros.org/wiki/xacro"  name="TTR01">
     <xacro:include filename="robot_parameters.xacro"/>
-    <!--base/world frame-->
-    <link name="base_link"> </link>
-    <!--Bottom base frame-->
-    <joint name="B_base_joint" type="fixed">
-        <origin xyz="0 0 0.05606" rpy="0 0 0"/>
-        <parent link="base_link"/>
-        <child link="B_base_link"/>
-    </joint>
-    <xacro:property name="B_base_length" value="0.005"/>
-    <xacro:property name="B_base_radius" value="0.089"/>
-    <link name="B_base_link">
-        <visual>
-            <origin xyz="0 0 -${B_base_length/2}" rpy="0 0 0"/>
-            <geometry>
-                <!--<mesh filename="package://robot_pkg/meshes/base_link.STL" />-->
-                <cylinder length="${B_base_length}" radius="${B_base_radius}"/>
-            </geometry>
-            <material name="white"/>
-        </visual>
-        <collision>
-            <origin xyz="0 0 -${B_base_length/2}" rpy="0 0 0"/>
-            <geometry>
-                <!--<mesh filename="package://robot_pkg/meshes/base_link.STL" />-->
-                <cylinder length="${B_base_length}" radius="${B_base_radius}"/>
-            </geometry>
-        </collision>
-        <xacro:inertial_cylinder mass="0.9" length="${B_base_length}" radius="${B_base_radius}">
-            <origin xyz="0 0 -${B_base_length/2}" rpy="0 0 0"/>
-        </xacro:inertial_cylinder>
-    </link>
-    <!--Left wheel frame-->
-    <joint name="L_wheel_joint" type="continuous">
-        <origin xyz="0 -0.10575 -0.02356" rpy="${pi/2} ${pi/2} 0"/>
-        <parent link="B_base_link"/>
-        <child link="L_wheel_link"/>
-        <axis xyz="0 0 1"/>
-        <limit effort="0.323" velocity="10.47" />
-    </joint>
-    <xacro:property name="wheel_thickness" value="0.027"/>
-    <xacro:property name="wheel_radius" value="0.0325"/>
-    <link name="L_wheel_link">
-        <visual>
-            <origin xyz="0 0 0" rpy="0 0 0"/>
-            <geometry>
-                <cylinder length="${wheel_thickness}" radius="${wheel_radius}"/>
-            </geometry>
-            <material name="black"/>
-        </visual>
-        <collision>
-            <origin xyz="0 0 0" rpy="0 0 0"/>
-            <geometry>
-                <cylinder length="${wheel_thickness}" radius="${wheel_radius}"/>
-            </geometry>
-        </collision>
-        <xacro:inertial_cylinder mass="0.05" length="${wheel_thickness}" radius="${wheel_radius}">
-            <origin xyz="0 0 0" rpy="0 0 0"/>
-        </xacro:inertial_cylinder>
-    </link>
-    <!--Right wheel frame-->
-    <joint name="R_wheel_joint" type="continuous">
-        <origin xyz="0 0.10575 -0.02356" rpy="${-pi/2} ${pi/2} 0"/>
-        <parent link="B_base_link"/>
-        <child link="R_wheel_link"/>
-        <axis xyz="0 0 -1"/>
-        <limit effort="0.323" velocity="10.47" />
-    </joint>
-    <link name="R_wheel_link">
-        <visual>
-            <origin xyz="0 0 0" rpy="0 0 0"/>
-            <geometry>
-                <cylinder length="${wheel_thickness}" radius="${wheel_radius}"/>
-            </geometry>
-            <material name="black"/>
-        </visual>
-        <collision>
-            <origin xyz="0 0 0" rpy="0 0 0"/>
-            <geometry>
-                <cylinder length="${wheel_thickness}" radius="${wheel_radius}"/>
-            </geometry>
-        </collision>
-        <xacro:inertial_cylinder mass="0.05" length="${wheel_thickness}" radius="${wheel_radius}">
-            <origin xyz="0 0 0" rpy="0 0 0"/>
-        </xacro:inertial_cylinder>
-    </link>
-    <!--Caster wheel base 1-->
-    <joint name="U_base_wheel_1_joint" type="continuous">
-        <origin xyz="0.05751 0 -0.0278" rpy="${pi} 0 0"/>
-        <parent link="B_base_link"/>
-        <child link="U_base_wheel_1_link"/>
-        <axis xyz="0 0 1"/>
-    </joint>
-    <xacro:property name="U_base_box_X" value="0.028"/>
-    <xacro:property name="U_base_box_Y" value="0.032"/>
-    <xacro:property name="U_base_box_Z" value="0.03902"/>
-    <link name="U_base_wheel_1_link">
-        <visual>
-            <origin xyz="0 0 -0.00329" rpy="0 0 0"/>
-            <geometry>
-                <box size="${U_base_box_X} ${U_base_box_Y} ${U_base_box_Z}"/>
-            </geometry>
-            <material name="light_gray"/>
-        </visual>
-        <collision>
-            <origin xyz="0 0 -0.00329" rpy="0 0 0"/>
-            <geometry>
-                <box size="${U_base_box_X} ${U_base_box_Y} ${U_base_box_Z}"/>
-            </geometry>
-        </collision>
-        <xacro:inertial_box mass="0.0125" x="${U_base_box_X}" y="${U_base_box_Y}" z="${U_base_box_Z}">
-            <origin xyz="0 0 0" rpy="0 0 0"/>
-        </xacro:inertial_box>
-    </link>
-    <!--Caster wheel 1-->
-    <joint name="U_wheel_1_joint" type="continuous">
-        <origin xyz="0.01577 0 0.01622" rpy="${pi/2} 0 0"/>
-        <parent link="U_base_wheel_1_link"/>
-        <child link="U_wheel_1_link"/>
-        <axis xyz="0 0 1"/>
-    </joint>
-    <xacro:property name="U_wheel_thickness" value="0.0144"/>
-    <xacro:property name="U_wheel_radius" value="0.0115"/>
-    <link name="U_wheel_1_link">
-        <visual>
-            <origin xyz="0 0 0" rpy="0 0 0"/>
-            <geometry>
-                <cylinder radius="${U_wheel_radius}" length="${U_wheel_thickness}"/>
-            </geometry>
-            <material name="white"/>
-        </visual>
-        <collision>
-            <origin xyz="0 0 0" rpy="0 0 0"/>
-            <geometry>
-                <cylinder radius="${U_wheel_radius}" length="${U_wheel_thickness}"/>
-            </geometry>
-        </collision>
-        <xacro:inertial_cylinder mass="0.005" length="${U_wheel_thickness}" radius="${U_wheel_radius}">
-            <origin xyz="0 0 0" rpy="0 0 0"/>
-        </xacro:inertial_cylinder>
-    </link>
-    <!--Caster wheel base 2-->
-    <joint name="U_base_wheel_2_joint" type="continuous">
-        <origin xyz="-0.05751 0 -0.0278" rpy="${pi} 0 ${pi}"/>
-        <parent link="B_base_link"/>
-        <child link="U_base_wheel_2_link"/>
-        <axis xyz="0 0 1"/>
-        <limit effort="0" velocity="0" />
-    </joint>
-    <link name="U_base_wheel_2_link">
-        <visual>
-            <origin xyz="0 0 -0.00329" rpy="0 0 0"/>
-            <geometry>
-                <box size="${U_base_box_X} ${U_base_box_Y} ${U_base_box_Z}"/>
-            </geometry>
-            <material name="light_gray"/>
-        </visual>
-        <collision>
-            <origin xyz="0 0 -0.00329" rpy="0 0 0"/>
-            <geometry>
-                <box size="${U_base_box_X} ${U_base_box_Y} ${U_base_box_Z}"/>
-            </geometry>
-        </collision>
-        <xacro:inertial_box mass="0.0125" x="${U_base_box_X}" y="${U_base_box_Y}" z="${U_base_box_Z}">
-            <origin xyz="0 0 0" rpy="0 0 0"/>
-        </xacro:inertial_box>
-    </link>
-    <!--Caster wheel 2-->
-    <joint name="U_wheel_2_joint" type="continuous">
-        <origin xyz="0.01577 0 0.01622" rpy="${pi/2} 0 0"/>
-        <parent link="U_base_wheel_2_link"/>
-        <child link="U_wheel_2_link"/>
-        <axis xyz="0 0 -1"/>
-        <limit effort="0" velocity="0" />
-    </joint>
-    <link name="U_wheel_2_link">
-        <visual>
-            <origin xyz="0 0 0" rpy="0 0 0"/>
-            <geometry>
-                <cylinder radius="${U_wheel_radius}" length="${U_wheel_thickness}"/>
-            </geometry>
-            <material name="white"/>
-        </visual>
-        <collision>
-            <origin xyz="0 0 0" rpy="0 0 0"/>
-            <geometry>
-                <cylinder radius="${U_wheel_radius}" length="${U_wheel_thickness}"/>
-            </geometry>
-        </collision>
-        <xacro:inertial_cylinder mass="0.005" length="${U_wheel_thickness}" radius="${U_wheel_radius}">
-            <origin xyz="0 0 0" rpy="0 0 0"/>
-        </xacro:inertial_cylinder>
-    </link>
-    <!--Fixed support-->
-    <joint name="Support_joint" type="fixed">
-        <origin xyz="0 0 0.101" rpy="0 0 0"/>
-        <parent link="B_base_link"/>
-        <child link="Support_link"/>
-    </joint>
-    <xacro:property name="Support_length" value="0.101"/>
-    <xacro:property name="Support_radius" value="0.070"/>
-    <link name="Support_link">
-        <visual>
-            <origin xyz="0 0 -${Support_length/2}" rpy="0 0 0"/>
-            <geometry>
-                <cylinder length="${Support_length}" radius="${Support_radius}"/>
-            </geometry>
-            <material name="white"/>
-        </visual>
-        <collision>
-            <origin xyz="0 0 -${Support_length/2}" rpy="0 0 0"/>
-            <geometry>
-                <cylinder length="${Support_length}" radius="${Support_radius}"/>
-            </geometry>
-        </collision>
-        <xacro:inertial_cylinder mass="0.5" length="${Support_length}" radius="${Support_radius}">
-            <origin xyz="0 0 -${Support_length/2}" rpy="0 0 0"/>
-        </xacro:inertial_cylinder>
-    </link>
+    <xacro:include filename="robot.xacro"/>
     <xacro:include filename="gazebo_setup.xacro"/>
 </robot>

File: src/robot_pkg/urdf/gazebo_setup.xacro (robot description, xacro)
@@ -32,5 +32,5 @@
                 <ode>
                     <mu>1.0</mu>
-                    <mu2>0.8</mu2>
+                    <mu2>1.0</mu2>
                 </ode>
             </friction>
@@ -42,5 +42,5 @@
                 <ode>
                     <mu>1.0</mu>
-                    <mu2>0.8</mu2>
+                    <mu2>1.0</mu2>
                 </ode>
             </friction>
@@ -52,6 +52,6 @@
           <friction>
               <ode>
-                  <mu>0.001</mu>
-                  <mu2>0.001</mu2>
+                  <mu>0.1</mu>
+                  <mu2>0.1</mu2>
               </ode>
           </friction>
@@ -72,6 +72,6 @@
       <friction>
           <ode>
-              <mu>0.001</mu>
-              <mu2>0.001</mu2>
+              <mu>0.1</mu>
+              <mu2>0.1</mu2>
           </ode>
       </friction>
@@ -116,5 +116,5 @@
             <!-- Limits -->
             <max_wheel_torque>0.5</max_wheel_torque>
-            <max_wheel_acceleration>43.15</max_wheel_acceleration>
+            <max_wheel_acceleration>10.47</max_wheel_acceleration>
             <!-- Output -->
             <odometry_frame>odom</odometry_frame>

File: src/robot_pkg/urdf/robot_parameters.xacro (robot description, xacro)
@@ -20,4 +20,22 @@
         <color rgba="0 0 0 1"/>
     </material>
+    <!--Measures-->
+    <xacro:property name="B_base_length" value="0.005"/>
+    <xacro:property name="B_base_radius" value="0.089"/>
+    <xacro:property name="wheel_thickness" value="0.027"/>
+    <xacro:property name="wheel_radius" value="0.0325"/>
+    <xacro:property name="U_base_box_X" value="0.028"/>
+    <xacro:property name="U_base_box_Y" value="0.032"/>
+    <xacro:property name="U_base_box_Z" value="0.03902"/>
+    <xacro:property name="U_wheel_thickness" value="0.0144"/>
+    <xacro:property name="U_wheel_radius" value="0.0115"/>
+    <xacro:property name="Support_length" value="0.101"/>
+    <xacro:property name="Support_radius" value="0.070"/>
+    <!--Mass-->
+    <xacro:property name="B_base_mass" value="1.0"/>
+    <xacro:property name="wheel_mass" value="0.120"/>
+    <xacro:property name="U_base_mass" value="0.05"/>
+    <xacro:property name="U_wheel_mass" value="0.01"/>
+    <xacro:property name="Support_mass" value="1.0"/>
     <!-- Standard inertial calculations https://en.wikipedia.org/wiki/List_of_moments_of_inertia -->
     <xacro:macro name="inertial_sphere" params="mass radius *origin">
@@ -35,5 +53,5 @@
             <mass value="${mass}" />
             <inertia ixx="${(1/12) * mass * (y*y+z*z)}" ixy="0.0" ixz="0.0"
-                    iyy="${(1/12) * mass * (x*x+z*z)}" iyz="0.0"
+                    iyy="${(1/12) * mass * (z*z+x*x)}" iyz="0.0"
                     izz="${(1/12) * mass * (x*x+y*y)}" />
         </inertial>

Commit message: lidar

File: src/robot_pkg/urdf/TTR01.urdf.xacro (robot description, xacro)
@@ -4,3 +4,4 @@
     <xacro:include filename="robot.xacro"/>
     <xacro:include filename="gazebo_setup.xacro"/>
+    <xacro:include filename="lidar.xacro"/>
 </robot>

File: src/robot_pkg/urdf/gazebo_setup.xacro (robot description, xacro)
@@ -24,4 +24,7 @@
     </gazebo>
     <gazebo reference="Support_link">
+      <material>Gazebo/White</material>
+    </gazebo>
+    <gazebo reference="Lidar_base_link">
       <material>Gazebo/White</material>
     </gazebo>
@@ -98,4 +101,5 @@
             <joint_name>U_base_wheel_2_joint</joint_name>
             <joint_name>U_wheel_2_joint</joint_name>
+             <joint_name>Lidar_motor_joint</joint_name>
         </plugin>
     </gazebo>

File: src/robot_pkg/urdf/robot_parameters.xacro (robot description, xacro)
@@ -32,4 +32,9 @@
     <xacro:property name="Support_length" value="0.101"/>
     <xacro:property name="Support_radius" value="0.070"/>
+    <xacro:property name="Lidar_base_X" value="0.10457"/>
+    <xacro:property name="Lidar_base_Y" value="0.0787"/>
+    <xacro:property name="Lidar_base_Z" value="0.0305"/>
+    <xacro:property name="Lidar_motor_length" value="0.0245"/>
+    <xacro:property name="Lidar_motor_radius" value="0.035"/>
     <!--Mass-->
     <xacro:property name="B_base_mass" value="1.0"/>
@@ -38,4 +43,6 @@
     <xacro:property name="U_wheel_mass" value="0.01"/>
     <xacro:property name="Support_mass" value="1.0"/>
+    <xacro:property name="Lidar_base_mass" value="0.1"/>
+    <xacro:property name="Lidar_motor_mass" value="0.1"/>
     <!-- Standard inertial calculations https://en.wikipedia.org/wiki/List_of_moments_of_inertia -->
     <xacro:macro name="inertial_sphere" params="mass radius *origin">
