Commit message: gazebo camera

File: src/robot_pkg/urdf/TTR01.urdf.xacro (robot description, xacro)
@@ -5,3 +5,4 @@
     <xacro:include filename="gazebo_setup.xacro"/>
     <xacro:include filename="lidar.xacro"/>
+    <xacro:include filename="camera.xacro" />
 </robot>

File: src/robot_pkg/urdf/gazebo_setup.xacro (robot description, xacro)
@@ -23,9 +23,24 @@
       <material>Gazebo/White</material>
     </gazebo>
-    <gazebo reference="Support_link">
+    <gazebo reference="Support_A_link">
+      <material>Gazebo/White</material>
+    </gazebo>
+    <gazebo reference="M_base_link">
+      <material>Gazebo/Black</material>
+    </gazebo>
+    <gazebo reference="Support_B_link">
+      <material>Gazebo/White</material>
+    </gazebo>
+    <gazebo reference="T_base_link">
       <material>Gazebo/White</material>
     </gazebo>
     <gazebo reference="Lidar_base_link">
       <material>Gazebo/White</material>
+    </gazebo>
+    <gazebo reference="Camera_base_link">
+      <material>Gazebo/Black</material>
+    </gazebo>
+    <gazebo reference="Camera_link">
+      <material>Gazebo/Green</material>
     </gazebo>
     <!-- Define friction for wheels -->

File: src/robot_pkg/urdf/lidar.xacro (robot description, xacro)
@@ -4,5 +4,5 @@
     <joint name="Lidar_base_joint" type="fixed">
         <origin xyz="0 0 0.0305" rpy="0 0 0"/>
-        <parent link="Support_link"/>
+        <parent link="T_base_link"/>
         <child link="Lidar_base_link"/>
     </joint>
@@ -53,5 +53,5 @@
         <sensor name="laser" type="ray">
             <pose> 0 0 0 0 0 0 </pose>
-            <visualize> true </visualize>
+            <visualize> false </visualize>
             <upadet_rate> 10 </upadet_rate>
             <ray>

File: src/robot_pkg/urdf/robot.xacro (robot description, xacro)
@@ -1,9 +1,9 @@
 <?xml version="1.0"?>
 <robot xmlns:xacro="http://www.ros.org/wiki/xacro" >
-    <!--base/world frame-->
+    <!--base/world-->
     <link name="base_link"> </link>
-    <!--Bottom base frame-->
+    <!--Bottom base-->
     <joint name="B_base_joint" type="fixed">
-        <origin xyz="0 0 0.05606" rpy="0 0 0"/>
+        <origin xyz="0 0 0.0225" rpy="0 0 0"/>
         <parent link="base_link"/>
         <child link="B_base_link"/>
@@ -29,10 +29,10 @@
         </xacro:inertial_cylinder>
     </link>
-    <!--Left wheel frame-->
+    <!--Left wheel-->
     <joint name="L_wheel_joint" type="continuous">
         <origin xyz="0 -0.10575 -0.02356" rpy="${pi/2} ${pi/2} 0"/>
         <parent link="B_base_link"/>
         <child link="L_wheel_link"/>
-        <axis xyz="0 0 1"/>
+        <axis xyz="0 0 -1"/>
         <limit effort="0.323" velocity="10.47" />
     </joint>
@@ -55,10 +55,10 @@
         </xacro:inertial_cylinder>
     </link>
-    <!--Right wheel frame-->
+    <!--Right wheel-->
     <joint name="R_wheel_joint" type="continuous">
         <origin xyz="0 0.10575 -0.02356" rpy="${-pi/2} ${pi/2} 0"/>
         <parent link="B_base_link"/>
         <child link="R_wheel_link"/>
-        <axis xyz="0 0 -1"/>
+        <axis xyz="0 0 1"/>
         <limit effort="0.323" velocity="10.47" />
     </joint>
@@ -111,5 +111,5 @@
         <parent link="U_base_wheel_1_link"/>
         <child link="U_wheel_1_link"/>
-        <axis xyz="0 0 1"/>
+        <axis xyz="0 0 -1"/>
     </joint>
     <link name="U_wheel_1_link">
@@ -136,5 +136,5 @@
         <parent link="B_base_link"/>
         <child link="U_base_wheel_2_link"/>
-        <axis xyz="0 0 1"/>
+        <axis xyz="0 0 -1"/>
     </joint>
     <link name="U_base_wheel_2_link">
@@ -161,5 +161,5 @@
         <parent link="U_base_wheel_2_link"/>
         <child link="U_wheel_2_link"/>
-        <axis xyz="0 0 -1"/>
+        <axis xyz="0 0 1"/>
     </joint>
     <link name="U_wheel_2_link">
@@ -181,26 +181,98 @@
         </xacro:inertial_cylinder>
     </link>
-    <!--Fixed support-->
-    <joint name="Support_joint" type="fixed">
-        <origin xyz="0 0 0.101" rpy="0 0 0"/>
-        <parent link="B_base_link"/>
-        <child link="Support_link"/>
-    </joint>
-    <link name="Support_link">
-        <visual>
-            <origin xyz="0 0 -${Support_length/2}" rpy="0 0 0"/>
-            <geometry>
-                <cylinder length="${Support_length}" radius="${Support_radius}"/>
-            </geometry>
-            <material name="white"/>
-        </visual>
-        <collision>
-            <origin xyz="0 0 -${Support_length/2}" rpy="0 0 0"/>
-            <geometry>
-                <cylinder length="${Support_length}" radius="${Support_radius}"/>
-            </geometry>
-        </collision>
-        <xacro:inertial_cylinder mass="${Support_mass}" length="${Support_length}" radius="${Support_radius}">
-            <origin xyz="0 0 -${Support_length/2}" rpy="0 0 0"/>
+    <!--Support A-->
+    <joint name="Support_A_joint" type="fixed">
+        <origin xyz="0 0 0.02" rpy="0 0 0"/>
+        <parent link="B_base_link"/>
+        <child link="Support_A_link"/>
+    </joint>
+    <link name="Support_A_link">
+        <visual>
+            <origin xyz="0 0 0" rpy="0 0 0"/>
+            <geometry>
+                <box size="${Support_AX} ${Support_AY} ${Support_AZ}"/>
+            </geometry>
+            <material name="white"/>
+        </visual>
+        <collision>
+            <origin xyz="0 0 0" rpy="0 0 0"/>
+            <geometry>
+                <box size="${Support_AX} ${Support_AY} ${Support_AZ}"/>
+            </geometry>
+        </collision>
+        <xacro:inertial_box mass="${Support_A_mass}" x="${Support_AX}" y="${Support_AY}" z="${Support_AZ}">
+            <origin xyz="0 0 0" rpy="0 0 0"/>
+        </xacro:inertial_box>
+    </link>
+    <!--Middle base-->
+    <joint name="M_base_joint" type="fixed">
+        <origin xyz="0 0 0.025" rpy="0 0 0"/>
+        <parent link="Support_A_link"/>
+        <child link="M_base_link"/>
+    </joint>
+    <link name="M_base_link">
+        <visual>
+            <origin xyz="0 0 -${MT_length/2}" rpy="0 0 0"/>
+            <geometry>
+                <cylinder length="${MT_length}" radius="${MT_radius}"/>
+            </geometry>
+            <material name="black"/>
+        </visual>
+        <collision>
+            <origin xyz="0 0 -${MT_length/2}" rpy="0 0 0"/>
+            <geometry>
+                <cylinder length="${MT_length}" radius="${MT_radius}"/>
+            </geometry>
+        </collision>
+        <xacro:inertial_cylinder mass="${MT_mass}" length="${MT_length}" radius="${MT_radius}">
+            <origin xyz="0 0 -${MT_length/2}" rpy="0 0 0"/>
+        </xacro:inertial_cylinder>
+    </link>
+    <!--Support B-->
+    <joint name="Support_B_joint" type="fixed">
+        <origin xyz="0 0 0.0255" rpy="0 0 0"/>
+        <parent link="M_base_link"/>
+        <child link="Support_B_link"/>
+    </joint>
+    <link name="Support_B_link">
+        <visual>
+            <origin xyz="0 0 0" rpy="0 0 0"/>
+            <geometry>
+                <box size="${Support_BX} ${Support_BY} ${Support_BZ}"/>
+            </geometry>
+            <material name="white"/>
+        </visual>
+        <collision>
+            <origin xyz="0 0 0" rpy="0 0 0"/>
+            <geometry>
+                <box size="${Support_BX} ${Support_BY} ${Support_BZ}"/>
+            </geometry>
+        </collision>
+        <xacro:inertial_box mass="${Support_B_mass}" x="${Support_BX}" y="${Support_BY}" z="${Support_AZ}">
+            <origin xyz="0 0 0" rpy="0 0 0"/>
+        </xacro:inertial_box>
+    </link>
+    <!--Top base-->
+    <joint name="T_base_joint" type="fixed">
+        <origin xyz="0 0 0.0305" rpy="0 0 0"/>
+        <parent link="Support_B_link"/>
+        <child link="T_base_link"/>
+    </joint>
+    <link name="T_base_link">
+        <visual>
+            <origin xyz="0 0 -${MT_length/2}" rpy="0 0 0"/>
+            <geometry>
+                <cylinder length="${MT_length}" radius="${MT_radius}"/>
+            </geometry>
+            <material name="white"/>
+        </visual>
+        <collision>
+            <origin xyz="0 0 -${MT_length/2}" rpy="0 0 0"/>
+            <geometry>
+                <cylinder length="${MT_length}" radius="${MT_radius}"/>
+            </geometry>
+        </collision>
+        <xacro:inertial_cylinder mass="${MT_mass}" length="${MT_length}" radius="${MT_radius}">
+            <origin xyz="0 0 -${MT_length/2}" rpy="0 0 0"/>
         </xacro:inertial_cylinder>
     </link>

File: src/robot_pkg/urdf/robot_parameters.xacro (robot description, xacro)
@@ -1,5 +1,5 @@
 <?xml version="1.0"?>
 <robot xmlns:xacro="http://www.ros.org/wiki/xacro" >
-    <!-- colors -->
+    <!-- Colors -->
     <material name="white">
         <color rgba="1 1 1 1"/>
@@ -10,4 +10,7 @@
     <material name="blue">
         <color rgba="0.2 0.2 1 1"/>
+    </material>
+    <material name="green">
+        <color rgba="0 0.8 0.1 1"/>
     </material>
     <material name="light_gray">
@@ -23,13 +26,19 @@
     <xacro:property name="B_base_length" value="0.005"/>
     <xacro:property name="B_base_radius" value="0.089"/>
+    <xacro:property name="MT_length" value="0.005"/>
+    <xacro:property name="MT_radius" value="0.070"/>
+    <xacro:property name="Support_AX" value="0.07571"/>
+    <xacro:property name="Support_AY" value="0.07648"/>
+    <xacro:property name="Support_AZ" value="0.04"/>
+    <xacro:property name="Support_BX" value="0.07571"/>
+    <xacro:property name="Support_BY" value="0.07648"/>
+    <xacro:property name="Support_BZ" value="0.051"/>
     <xacro:property name="wheel_thickness" value="0.027"/>
     <xacro:property name="wheel_radius" value="0.0325"/>
-    <xacro:property name="U_base_box_X" value="0.028"/>
-    <xacro:property name="U_base_box_Y" value="0.032"/>
+    <xacro:property name="U_base_box_X" value="0.032"/>
+    <xacro:property name="U_base_box_Y" value="0.038"/>
     <xacro:property name="U_base_box_Z" value="0.03902"/>
     <xacro:property name="U_wheel_thickness" value="0.0144"/>
     <xacro:property name="U_wheel_radius" value="0.0115"/>
-    <xacro:property name="Support_length" value="0.101"/>
-    <xacro:property name="Support_radius" value="0.070"/>
     <xacro:property name="Lidar_base_X" value="0.10457"/>
     <xacro:property name="Lidar_base_Y" value="0.0787"/>
@@ -37,12 +46,22 @@
     <xacro:property name="Lidar_motor_length" value="0.0245"/>
     <xacro:property name="Lidar_motor_radius" value="0.035"/>
+    <xacro:property name="Camera_base_X" value="0.0265"/>
+    <xacro:property name="Camera_base_Y" value="0.0335"/>
+    <xacro:property name="Camera_base_Z" value="0.01878"/>
+    <xacro:property name="Camera_X" value="0.00112"/>
+    <xacro:property name="Camera_Y" value="0.0246"/>
+    <xacro:property name="Camera_Z" value="0.024"/>
     <!--Mass-->
-    <xacro:property name="B_base_mass" value="1.0"/>
+    <xacro:property name="B_base_mass" value="0.08"/>
+    <xacro:property name="MT_mass" value="0.04"/>
+    <xacro:property name="Support_A_mass" value="0.3"/>
+    <xacro:property name="Support_B_mass" value="0.5"/>
     <xacro:property name="wheel_mass" value="0.120"/>
     <xacro:property name="U_base_mass" value="0.05"/>
     <xacro:property name="U_wheel_mass" value="0.01"/>
-    <xacro:property name="Support_mass" value="1.0"/>
     <xacro:property name="Lidar_base_mass" value="0.1"/>
     <xacro:property name="Lidar_motor_mass" value="0.1"/>
+    <xacro:property name="Camera_base_mass" value="0.025"/>
+    <xacro:property name="Camera_mass" value="0.01"/>
     <!-- Standard inertial calculations https://en.wikipedia.org/wiki/List_of_moments_of_inertia -->
     <xacro:macro name="inertial_sphere" params="mass radius *origin">

Commit message: control

File: src/robot_pkg/urdf/TTR01.urdf.xacro (robot description, xacro)
@@ -4,7 +4,7 @@
     <xacro:include filename="robot.xacro"/>
     <xacro:include filename="gazebo_setup.xacro"/>
-    <!-- <xacro:include filename="gazebo_control.xacro"/> -->
     <xacro:include filename="lidar.xacro"/>
     <xacro:include filename="camera.xacro" />
     <xacro:include filename="ros2_control.xacro" />
+    <!-- <xacro:include filename="gazebo_control.xacro"/> -->
 </robot>

File: src/robot_pkg/urdf/gazebo_setup.xacro (robot description, xacro)
@@ -66,5 +66,5 @@
     </gazebo>
     <!-- Define friction for caster wheels -->
-    <gazebo reference="U_base_wheel_1_joint">
+    <!-- <gazebo reference="U_base_wheel_1_joint">
       <surface>
           <friction>
@@ -75,5 +75,5 @@
           </friction>
       </surface>
-  </gazebo>
+  </gazebo> -->
   <gazebo reference="U_wheel_1_joint">
     <surface>
@@ -86,5 +86,5 @@
     </surface>
 </gazebo>
-<gazebo reference="U_base_wheel_2_joint">
+<!-- <gazebo reference="U_base_wheel_2_joint">
   <surface>
       <friction>
@@ -95,5 +95,5 @@
       </friction>
   </surface>
-</gazebo>
+</gazebo> -->
 <gazebo reference="U_wheel_2_joint">
 <surface>
@@ -112,8 +112,8 @@
             <joint_name>L_wheel_joint</joint_name>
             <joint_name>R_wheel_joint</joint_name>
-            <joint_name>U_base_wheel_1_joint</joint_name>
+            <!-- <joint_name>U_base_wheel_1_joint</joint_name>
             <joint_name>U_wheel_1_joint</joint_name>
             <joint_name>U_base_wheel_2_joint</joint_name>
-            <joint_name>U_wheel_2_joint</joint_name>
+            <joint_name>U_wheel_2_joint</joint_name> -->
              <joint_name>Lidar_motor_joint</joint_name>
         </plugin>

File: src/robot_pkg/urdf/robot.xacro (robot description, xacro)
@@ -82,9 +82,9 @@
     </link>
     <!--Caster wheel base 1-->
-    <joint name="U_base_wheel_1_joint" type="continuous">
+    <joint name="U_base_wheel_1_joint" type="fixed">
         <origin xyz="0.05751 0 -0.0278" rpy="${pi} 0 0"/>
         <parent link="B_base_link"/>
         <child link="U_base_wheel_1_link"/>
-        <axis xyz="0 0 1"/>
+        <!-- <axis xyz="0 0 1"/> -->
     </joint>
     <link name="U_base_wheel_1_link">
@@ -107,9 +107,9 @@
     </link>
     <!--Caster wheel 1-->
-    <joint name="U_wheel_1_joint" type="continuous">
+    <joint name="U_wheel_1_joint" type="fixed">
         <origin xyz="0.01577 0 0.01622" rpy="${pi/2} 0 0"/>
         <parent link="U_base_wheel_1_link"/>
         <child link="U_wheel_1_link"/>
-        <axis xyz="0 0 -1"/>
+        <!-- <axis xyz="0 0 -1"/>    -->
     </joint>
     <link name="U_wheel_1_link">
@@ -132,9 +132,9 @@
     </link>
     <!--Caster wheel base 2-->
-    <joint name="U_base_wheel_2_joint" type="continuous">
+    <joint name="U_base_wheel_2_joint" type="fixed">
         <origin xyz="-0.05751 0 -0.0278" rpy="${pi} 0 ${pi}"/>
         <parent link="B_base_link"/>
         <child link="U_base_wheel_2_link"/>
-        <axis xyz="0 0 -1"/>
+        <!-- <axis xyz="0 0 -1"/> -->
     </joint>
     <link name="U_base_wheel_2_link">
@@ -157,9 +157,9 @@
     </link>
     <!--Caster wheel 2-->
-    <joint name="U_wheel_2_joint" type="continuous">
+    <joint name="U_wheel_2_joint" type="fixed">
         <origin xyz="0.01577 0 0.01622" rpy="${pi/2} 0 0"/>
         <parent link="U_base_wheel_2_link"/>
         <child link="U_wheel_2_link"/>
-        <axis xyz="0 0 1"/>
+        <!-- <axis xyz="0 0 1"/>   -->
     </joint>
     <link name="U_wheel_2_link">

File: src/robot_pkg/urdf/ros2_control.xacro (robot description, xacro)
@@ -1,5 +1,33 @@
 <?xml version="1.0"?>
 <robot xmlns:xacro="http://www.ros.org/wiki/xacro">
-    <ros2_control name="GazeboSystem" type="system">
+    <ros2_control name="RealRobot" type="system">
+        <hardware>
+            <plugin>diffdrive_arduino/DiffDriveArduino</plugin>
+            <param name="left_wheel_name">L_wheel_joint</param>
+            <param name="right_wheel_name">R_wheel_joint</param>
+            <param name="loop_rate">30</param>
+            <param name="device">/dev/ttyUSB1</param>
+            <param name="baud_rate">57600</param>
+            <param name="timeout">1400</param>
+            <param name="enc_counts_per_rev">2491</param>
+        </hardware>
+        <joint name="L_wheel_joint">
+            <command_interface name="velocity">
+                <param name="min">-10</param>
+                <param name="max">10</param>
+            </command_interface>
+            <state_interface name="velocity"/>
+            <state_interface name="position"/>
+        </joint>
+        <joint name="L_wheel_joint">
+            <command_interface name="velocity">
+                <param name="min">-10</param>
+                <param name="max">10</param>
+            </command_interface>
+            <state_interface name="velocity"/>
+            <state_interface name="position"/>
+        </joint>
+    </ros2_control>
+    <!-- <ros2_control name="GazeboSystem" type="system">
         <hardware>
             <plugin>gazebo_ros2_control/GazeboSystem</plugin>
@@ -26,5 +54,5 @@
                 <parameters> $(find robot_pkg)/config/controllers.yaml </parameters>
             </plugin>
-    </gazebo>
+    </gazebo> -->
     <!-- ros2 run controller_manager_ros_control_node -->
 </robot>
