Commit message: wheel drift

File: src/robot_pkg/urdf/robot.xacro (robot description, xacro)
@@ -48,5 +48,6 @@
             <origin xyz="0 0 0" rpy="0 0 0"/>
             <geometry>
-                <cylinder length="${wheel_thickness}" radius="${wheel_radius}"/>
+                <sphere radius="${wheel_radius}"/>
+                <!-- <cylinder length="${wheel_thickness}" radius="${wheel_radius}"/> -->
             </geometry>
         </collision>
@@ -74,5 +75,5 @@
             <origin xyz="0 0 0" rpy="0 0 0"/>
             <geometry>
-                <cylinder length="${wheel_thickness}" radius="${wheel_radius}"/>
+                <sphere radius="${wheel_radius}"/>
             </geometry>
         </collision>
