Commit message: slam

File: src/robot_pkg/urdf/lidar.xacro (robot description, xacro)
@@ -26,9 +26,8 @@
     </link>
     <!--Lidar motor frame-->
-    <joint name="Lidar_motor_joint" type="continuous">
+    <joint name="Lidar_motor_joint" type="fixed">
         <origin xyz="-0.011 0 0.01225" rpy="0 0 0"/>
         <parent link="Lidar_base_link"/>
         <child link="Lidar_motor_link"/>
-        <axis xyz="0 0 -1"/>
     </joint>
     <link name="Lidar_motor_link">
@@ -54,6 +53,7 @@
         <sensor name="laser" type="ray">
             <pose> 0 0 0 0 0 0 </pose>
-            <visualize> false </visualize>
-            <upadet_rate> 10 </upadet_rate>
+            <always_on>true</always_on>
+            <visualize> true </visualize>
+            <update_rate> 10 </update_rate>
             <ray>
                 <scan>
@@ -65,4 +65,9 @@
                     </horizontal>
                 </scan>
+                <noise>
+                    <type>gaussian</type>
+                    <mean>0.0</mean>
+                    <stddev>0.01</stddev>
+                </noise>
                 <range>
                     <min> 0.1 </min>

File: src/robot_pkg/urdf/robot.xacro (robot description, xacro)
@@ -3,4 +3,12 @@
     <!--base link-->
     <link name="base_link"> </link>
+    <!--Base footprint-->
+    <joint name="base_footprint_joint" type="fixed">
+        <origin xyz="0 0 -0.0341" rpy="0 0 0"/>
+        <parent link="base_link"/>
+        <child link="base_footprint"/>
+    </joint>
+    <link name="base_footprint">
+    </link>
     <!--Bottom base-->
     <joint name="B_base_joint" type="fixed">
@@ -76,4 +84,5 @@
             <geometry>
                 <sphere radius="${wheel_radius}"/>
+                <!-- <cylinder length="${wheel_thickness}" radius="${wheel_radius}"/> -->
             </geometry>
         </collision>
